Commit message: simulation stuff

File: maelstrom_description/urdf/base.xacro (robot description, xacro)
@@ -36,4 +36,14 @@
       <selfCollide>false</selfCollide>
     </gazebo>
+    <gazebo reference="${namespace}/base_link">
+      <visual>
+        <material>
+          <script>
+              <name>maelstrom/supreme</name>
+              <uri>$(find maelstrom_description)/meshes/maelstrom/scripts/supreme.material</uri>
+          </script>
+        </material>
+      </visual>
+    </gazebo>
     <!-- Set up hydrodynamic plugin given as input parameter -->
     <xacro:insert_block name="gazebo"/>

File: maelstrom_description/urdf/sensors.xacro (robot description, xacro)
@@ -7,3 +7,170 @@
     more examples or add you own custom sensor units.
   -->
+  <xacro:macro name="default_camera" params="namespace parent_link suffix *origin">
+    <xacro:regular_camera_plugin_macro
+      namespace="${namespace}"
+      suffix="${suffix}"
+      parent_link="${parent_link}"
+      topic="camera"
+      mass="0.1"
+      update_rate="30"
+      hfov="1.5125"
+      width="768"
+      height="492"
+      stddev="0.02"
+      scale="1.0">
+      <inertia ixx="0.00001" ixy="0.0" ixz="0.0" iyy="0.00001" iyz="0.0" izz="0.00001" />
+      <xacro:insert_block name="origin" />
+    </xacro:regular_camera_plugin_macro>
+  </xacro:macro>
+  <xacro:macro name="regular_camera_plugin_macro"
+    params="namespace suffix parent_link topic mass update_rate
+      hfov width height stddev scale
+      *inertia *origin">
+    <!-- Sensor link -->
+    <link name="${namespace}/camera${suffix}_link">
+      <inertial>
+        <xacro:insert_block name="inertia" />
+        <mass value="${mass}" />
+        <origin xyz="0 0 0" rpy="0 0 0" />
+      </inertial>
+      <visual>
+        <geometry>
+          <mesh filename="file://$(find uuv_sensor_ros_plugins)/meshes/oe14-372.dae" scale="${scale} ${scale} ${scale}"/>
+        </geometry>
+      </visual>
+      <xacro:no_collision/>
+    </link>
+    <joint name="${namespace}/camera${suffix}_joint" type="revolute">
+      <xacro:insert_block name="origin" />
+      <parent link="${parent_link}" />
+      <child link="${namespace}/camera${suffix}_link" />
+      <limit upper="0" lower="0" effort="0" velocity="0" />
+      <axis xyz="1 0 0"/>
+    </joint>
+    <link name="${namespace}/camera${suffix}_link_optical">
+      <xacro:box_inertial x="0.0001" y="0.0001" z="0.0001" mass="0.001">
+        <origin xyz="0 0 0" rpy="0 0 0"/>
+      </xacro:box_inertial>
+      <collision>
+        <!-- todo: gazebo needs a collision volume or it will ignore the pose of
+           the joint that leads to this link (and assume it to be the identity) -->
+        <geometry>
+          <cylinder length="0.000001" radius="0.000001"/>
+        </geometry>
+        <origin xyz="0 0 0" rpy="0 ${0.5*pi} 0"/>
+      </collision>
+    </link>
+    <joint name="${namespace}/camera${suffix}_optical_joint" type="revolute">
+      <origin xyz="0 0 0" rpy="${-pi/2} 0 ${-pi/2}"/>
+      <parent link="${namespace}/camera${suffix}_link"/>
+      <child link="${namespace}/camera${suffix}_link_optical"/>
+      <limit upper="0" lower="0" effort="0" velocity="0" />
+      <axis xyz="1 0 0"/>
+    </joint>
+    <gazebo reference="${namespace}/camera${suffix}_link">
+      <sensor type="camera" name="camera${suffix}">
+        <update_rate>${update_rate}</update_rate>
+        <camera name="camera${suffix}">
+          <horizontal_fov>${hfov}</horizontal_fov>
+          <image>
+            <width>${width}</width>
+            <height>${height}</height>
+            <format>R8G8B8</format>
+          </image>
+          <clip>
+            <near>0.05</near>
+            <far>3000</far>
+          </clip>
+          <noise>
+            <type>gaussian</type>
+            <mean>0.0</mean>
+            <stddev>${stddev}</stddev>
+          </noise>
+        </camera>
+        <plugin name="camera${suffix}_controller" filename="libgazebo_ros_camera.so">
+          <updateRate>${update_rate}</updateRate>
+          <cameraName>${namespace}/camera${suffix}</cameraName>
+          <frameName>camera${suffix}_link_optical</frameName>
+          <attenuationR>0.0</attenuationR>
+          <attenuationG>0.0</attenuationG>
+          <attenuationB>0.0</attenuationB>
+          <backgroundR>0</backgroundR>
+          <backgroundG>0</backgroundG>
+          <backgroundB>0</backgroundB>
+          <!-- required for ros depth cam -->
+          <imageTopicName>${topic}_image</imageTopicName>
+          <pointCloudTopicName>${topic}_cloud</pointCloudTopicName>
+          <depthImageTopicName>${topic}_depth</depthImageTopicName>
+          <depthImageCameraInfoTopicName>${topic}_depth_info</depthImageCameraInfoTopicName>
+          <pointCloudCutoff>10.0</pointCloudCutoff>
+        </plugin>
+      </sensor>
+    </gazebo>
+  </xacro:macro>
+  <xacro:macro name="underwater_camera_plugin_macro"
+    params="namespace suffix parent_link topic mass update_rate
+      hfov width height stddev
+      *inertia *origin">
+    <!-- Sensor link -->
+    <link name="${namespace}/camera${suffix}_link">
+      <inertial>
+        <xacro:insert_block name="inertia" />
+        <mass value="${mass}" />
+        <origin xyz="0 0 0" rpy="0 0 0" />
+      </inertial>
+      <visual>
+        <geometry>
+          <mesh filename="file://$(find uuv_sensor_ros_plugins)/meshes/oe14-372.dae" scale="1 1 1"/>
+        </geometry>
+      </visual>
+      <xacro:no_collision/>
+    </link>
+    <joint name="${namespace}/camera${suffix}_joint" type="revolute">
+      <xacro:insert_block name="origin" />
+      <parent link="${parent_link}" />
+      <child link="${namespace}/camera${suffix}_link" />
+      <axis xyz="1 0 0"/>
+      <limit upper="0" lower="0" effort="0" velocity="0" />
+    </joint>
+    <gazebo reference="${namespace}/camera${suffix}_link">
+      <sensor type="depth" name="camera${suffix}">
+        <update_rate>${update_rate}</update_rate>
+        <camera name="camera${suffix}">
+          <horizontal_fov>${hfov}</horizontal_fov>
+          <image>
+            <width>${width}</width>
+            <height>${height}</height>
+            <format>R8G8B8</format>
+          </image>
+          <clip>
+            <near>0.1</near>
+            <far>3000</far>
+          </clip>
+          <noise>
+            <type>gaussian</type>
+            <mean>0.0</mean>
+            <stddev>${stddev}</stddev>
+          </noise>
+        </camera>
+        <plugin name="camera${suffix}_controller" filename="libuuv_gazebo_ros_camera_plugin.so">
+          <updateRate>${update_rate}</updateRate>
+          <cameraName>${namespace}/camera${suffix}</cameraName>
+          <frameName>${namespace}/camera${suffix}_link</frameName>
+          <attenuationR>0.01</attenuationR>
+          <attenuationG>0.01</attenuationG>
+          <attenuationB>0.003</attenuationB>
+          <backgroundR>0</backgroundR>
+          <backgroundG>0</backgroundG>
+          <backgroundB>0</backgroundB>
+          <!-- required for ros depth cam -->
+          <imageTopicName>${topic}_image</imageTopicName>
+          <pointCloudTopicName>${topic}_cloud</pointCloudTopicName>
+          <depthImageTopicName>${topic}_depth</depthImageTopicName>
+          <depthImageCameraInfoTopicName>${topic}_depth_info</depthImageCameraInfoTopicName>
+          <pointCloudCutoff>10.0</pointCloudCutoff>
+        </plugin>
+      </sensor>
+    </gazebo>
+  </xacro:macro>
 </robot>

Commit message: sensors and mesh

File: maelstrom_description/urdf/base.xacro (robot description, xacro)
@@ -36,5 +36,5 @@
       <selfCollide>false</selfCollide>
     </gazebo>
-    <gazebo reference="${namespace}/base_link">
+    <!--<gazebo reference="${namespace}/base_link">
       <visual>
         <material>
@@ -45,5 +45,5 @@
         </material>
       </visual>
-    </gazebo>
+    </gazebo> -->
     <!-- Set up hydrodynamic plugin given as input parameter -->
     <xacro:insert_block name="gazebo"/>

File: maelstrom_description/urdf/properties.xacro (robot description, xacro)
@@ -47,4 +47,7 @@
     <xacro:property name="vsf_pos"><origin xyz="0.41921 -0.30628 0.10615" rpy="0 0 ${pi/4}" /></xacro:property>
     <xacro:property name="vsa_pos"><origin xyz="-0.37225 -0.30628 0.10615" rpy="0 0 ${-pi/4}" /></xacro:property>
+    <xacro:property name="forward_camera_R_pos"><origin xyz="0.3818 0.05038 0.11999" rpy="0 0 0" /></xacro:property>
+    <xacro:property name="forward_camera_L_pos"><origin xyz="0.3818 -0.05038 0.11999" rpy="0 0 0" /></xacro:property>
+    <xacro:property name="downward_camera_pos"><origin xyz="0.0711 0.0004 0" rpy="0 ${pi/2} 0" /></xacro:property>
     <!--
     Visual mesh file for the vehicle, usually in DAE (Collada) format. Be sure to store the
@@ -53,5 +56,5 @@
     Open the meshes for the RexROV vehicle in Blender to see an example on the mesh placement.
     -->
-    <xacro:property name="visual_mesh_file" value="file://$(find maelstrom_description)/meshes/maelstrom.dae"/>
+    <xacro:property name="visual_mesh_file" value="file://$(find maelstrom_description)/meshes/maelstromColored.dae"/>
     <!-- Collision geometry mesh, usually in STL format (it is recommended to keep
     this geometry as simple as possible to improve the performance the physics engine

File: maelstrom_description/urdf/sensors.xacro (robot description, xacro)
@@ -7,11 +7,10 @@
     more examples or add you own custom sensor units.
   -->
-  <xacro:macro name="default_camera" params="namespace parent_link suffix *origin">
-    <xacro:regular_camera_plugin_macro
-      namespace="${namespace}"
-      suffix="${suffix}"
-      parent_link="${parent_link}"
+<xacro:regular_camera_plugin_macro
+      namespace="sensors"
+      suffix="_forward_R"
+      parent_link="${namespace}/base_link"
       topic="camera"
-      mass="0.1"
+      mass="0.001"
       update_rate="30"
       hfov="1.5125"
@@ -21,156 +20,35 @@
       scale="1.0">
       <inertia ixx="0.00001" ixy="0.0" ixz="0.0" iyy="0.00001" iyz="0.0" izz="0.00001" />
-      <xacro:insert_block name="origin" />
-    </xacro:regular_camera_plugin_macro>
-  </xacro:macro>
-  <xacro:macro name="regular_camera_plugin_macro"
-    params="namespace suffix parent_link topic mass update_rate
-      hfov width height stddev scale
-      *inertia *origin">
-    <!-- Sensor link -->
-    <link name="${namespace}/camera${suffix}_link">
-      <inertial>
-        <xacro:insert_block name="inertia" />
-        <mass value="${mass}" />
-        <origin xyz="0 0 0" rpy="0 0 0" />
-      </inertial>
-      <visual>
-        <geometry>
-          <mesh filename="file://$(find uuv_sensor_ros_plugins)/meshes/oe14-372.dae" scale="${scale} ${scale} ${scale}"/>
-        </geometry>
-      </visual>
-      <xacro:no_collision/>
-    </link>
-    <joint name="${namespace}/camera${suffix}_joint" type="revolute">
-      <xacro:insert_block name="origin" />
-      <parent link="${parent_link}" />
-      <child link="${namespace}/camera${suffix}_link" />
-      <limit upper="0" lower="0" effort="0" velocity="0" />
-      <axis xyz="1 0 0"/>
-    </joint>
-    <link name="${namespace}/camera${suffix}_link_optical">
-      <xacro:box_inertial x="0.0001" y="0.0001" z="0.0001" mass="0.001">
-        <origin xyz="0 0 0" rpy="0 0 0"/>
-      </xacro:box_inertial>
-      <collision>
-        <!-- todo: gazebo needs a collision volume or it will ignore the pose of
-           the joint that leads to this link (and assume it to be the identity) -->
-        <geometry>
-          <cylinder length="0.000001" radius="0.000001"/>
-        </geometry>
-        <origin xyz="0 0 0" rpy="0 ${0.5*pi} 0"/>
-      </collision>
-    </link>
-    <joint name="${namespace}/camera${suffix}_optical_joint" type="revolute">
-      <origin xyz="0 0 0" rpy="${-pi/2} 0 ${-pi/2}"/>
-      <parent link="${namespace}/camera${suffix}_link"/>
-      <child link="${namespace}/camera${suffix}_link_optical"/>
-      <limit upper="0" lower="0" effort="0" velocity="0" />
-      <axis xyz="1 0 0"/>
-    </joint>
-    <gazebo reference="${namespace}/camera${suffix}_link">
-      <sensor type="camera" name="camera${suffix}">
-        <update_rate>${update_rate}</update_rate>
-        <camera name="camera${suffix}">
-          <horizontal_fov>${hfov}</horizontal_fov>
-          <image>
-            <width>${width}</width>
-            <height>${height}</height>
-            <format>R8G8B8</format>
-          </image>
-          <clip>
-            <near>0.05</near>
-            <far>3000</far>
-          </clip>
-          <noise>
-            <type>gaussian</type>
-            <mean>0.0</mean>
-            <stddev>${stddev}</stddev>
-          </noise>
-        </camera>
-        <plugin name="camera${suffix}_controller" filename="libgazebo_ros_camera.so">
-          <updateRate>${update_rate}</updateRate>
-          <cameraName>${namespace}/camera${suffix}</cameraName>
-          <frameName>camera${suffix}_link_optical</frameName>
-          <attenuationR>0.0</attenuationR>
-          <attenuationG>0.0</attenuationG>
-          <attenuationB>0.0</attenuationB>
-          <backgroundR>0</backgroundR>
-          <backgroundG>0</backgroundG>
-          <backgroundB>0</backgroundB>
-          <!-- required for ros depth cam -->
-          <imageTopicName>${topic}_image</imageTopicName>
-          <pointCloudTopicName>${topic}_cloud</pointCloudTopicName>
-          <depthImageTopicName>${topic}_depth</depthImageTopicName>
-          <depthImageCameraInfoTopicName>${topic}_depth_info</depthImageCameraInfoTopicName>
-          <pointCloudCutoff>10.0</pointCloudCutoff>
-        </plugin>
-      </sensor>
-    </gazebo>
-  </xacro:macro>
-  <xacro:macro name="underwater_camera_plugin_macro"
-    params="namespace suffix parent_link topic mass update_rate
-      hfov width height stddev
-      *inertia *origin">
-    <!-- Sensor link -->
-    <link name="${namespace}/camera${suffix}_link">
-      <inertial>
-        <xacro:insert_block name="inertia" />
-        <mass value="${mass}" />
-        <origin xyz="0 0 0" rpy="0 0 0" />
-      </inertial>
-      <visual>
-        <geometry>
-          <mesh filename="file://$(find uuv_sensor_ros_plugins)/meshes/oe14-372.dae" scale="1 1 1"/>
-        </geometry>
-      </visual>
-      <xacro:no_collision/>
-    </link>
-    <joint name="${namespace}/camera${suffix}_joint" type="revolute">
-      <xacro:insert_block name="origin" />
-      <parent link="${parent_link}" />
-      <child link="${namespace}/camera${suffix}_link" />
-      <axis xyz="1 0 0"/>
-      <limit upper="0" lower="0" effort="0" velocity="0" />
-    </joint>
-    <gazebo reference="${namespace}/camera${suffix}_link">
-      <sensor type="depth" name="camera${suffix}">
-        <update_rate>${update_rate}</update_rate>
-        <camera name="camera${suffix}">
-          <horizontal_fov>${hfov}</horizontal_fov>
-          <image>
-            <width>${width}</width>
-            <height>${height}</height>
-            <format>R8G8B8</format>
-          </image>
-          <clip>
-            <near>0.1</near>
-            <far>3000</far>
-          </clip>
-          <noise>
-            <type>gaussian</type>
-            <mean>0.0</mean>
-            <stddev>${stddev}</stddev>
-          </noise>
-        </camera>
-        <plugin name="camera${suffix}_controller" filename="libuuv_gazebo_ros_camera_plugin.so">
-          <updateRate>${update_rate}</updateRate>
-          <cameraName>${namespace}/camera${suffix}</cameraName>
-          <frameName>${namespace}/camera${suffix}_link</frameName>
-          <attenuationR>0.01</attenuationR>
-          <attenuationG>0.01</attenuationG>
-          <attenuationB>0.003</attenuationB>
-          <backgroundR>0</backgroundR>
-          <backgroundG>0</backgroundG>
-          <backgroundB>0</backgroundB>
-          <!-- required for ros depth cam -->
-          <imageTopicName>${topic}_image</imageTopicName>
-          <pointCloudTopicName>${topic}_cloud</pointCloudTopicName>
-          <depthImageTopicName>${topic}_depth</depthImageTopicName>
-          <depthImageCameraInfoTopicName>${topic}_depth_info</depthImageCameraInfoTopicName>
-          <pointCloudCutoff>10.0</pointCloudCutoff>
-        </plugin>
-      </sensor>
-    </gazebo>
-  </xacro:macro>
+      <xacro:insert_block name="forward_camera_R_pos" />
+</xacro:regular_camera_plugin_macro>
+<xacro:regular_camera_plugin_macro
+      namespace="sensors"
+      suffix="_forward_L"
+      parent_link="${namespace}/base_link"
+      topic="camera"
+      mass="0.001"
+      update_rate="30"
+      hfov="1.5125"
+      width="768"
+      height="492"
+      stddev="0.02"
+      scale="1.0">
+      <inertia ixx="0.00001" ixy="0.0" ixz="0.0" iyy="0.00001" iyz="0.0" izz="0.00001" />
+      <xacro:insert_block name="forward_camera_L_pos" />
+</xacro:regular_camera_plugin_macro>
+<xacro:regular_camera_plugin_macro
+      namespace="sensors"
+      suffix="_downward"
+      parent_link="${namespace}/base_link"
+      topic="camera"
+      mass="0.001"
+      update_rate="30"
+      hfov="1.5125"
+      width="768"
+      height="492"
+      stddev="0.02"
+      scale="1.0">
+      <inertia ixx="0.00001" ixy="0.0" ixz="0.0" iyy="0.00001" iyz="0.0" izz="0.00001" />
+      <xacro:insert_block name="downward_camera_pos" />
+</xacro:regular_camera_plugin_macro>
 </robot>

Commit message: Added sensors, quat_to_euler

File: maelstrom_description/urdf/base.xacro (robot description, xacro)
@@ -36,14 +36,4 @@
       <selfCollide>false</selfCollide>
     </gazebo>
-    <!--<gazebo reference="${namespace}/base_link">
-      <visual>
-        <material>
-          <script>
-              <name>maelstrom/supreme</name>
-              <uri>$(find maelstrom_description)/meshes/maelstrom/scripts/supreme.material</uri>
-          </script>
-        </material>
-      </visual>
-    </gazebo> -->
     <!-- Set up hydrodynamic plugin given as input parameter -->
     <xacro:insert_block name="gazebo"/>

File: maelstrom_description/urdf/sensors.xacro (robot description, xacro)
@@ -7,4 +7,5 @@
     more examples or add you own custom sensor units.
   -->
+<!-- right forward camerea-->
 <xacro:regular_camera_plugin_macro
       namespace="sensors"
@@ -22,4 +23,5 @@
       <xacro:insert_block name="forward_camera_R_pos" />
 </xacro:regular_camera_plugin_macro>
+<!-- left forward camera-->
 <xacro:regular_camera_plugin_macro
       namespace="sensors"
@@ -37,4 +39,5 @@
       <xacro:insert_block name="forward_camera_L_pos" />
 </xacro:regular_camera_plugin_macro>
+<!-- downward camera-->
 <xacro:regular_camera_plugin_macro
       namespace="sensors"
@@ -52,3 +55,21 @@
       <xacro:insert_block name="downward_camera_pos" />
 </xacro:regular_camera_plugin_macro>
+<!-- IMU -->
+<xacro:default_imu_macro
+      namespace="${namespace}"
+      parent_link="${namespace}/base_link"
+      inertial_reference_frame="world_ned">
+      <origin xyz="0 0 0" rpy="0 0 0"/>
+</xacro:default_imu_macro>
+<!--DVL-->
+<xacro:default_dvl_macro
+      namespace="${namespace}"
+      parent_link="${namespace}/base_link"
+      inertial_reference_frame="world_ned">
+      <origin xyz="-0.081297 -0.081297 0.0" rpy="0 ${0.5*pi} 0"/>
+</xacro:default_dvl_macro>
+<!--Depth Sensor-->
+<xacro:default_pressure_macro namespace="${namespace}" parent_link="${namespace}/base_link">
+      <origin xyz="0 -0.0004 0.0711" rpy="0 0 0"/>
+</xacro:default_pressure_macro>
 </robot>
