Commit message: Stable

File: maelstrom_description/urdf/properties.xacro (robot description, xacro)
@@ -2,5 +2,5 @@
 <robot xmlns:xacro="http://www.ros.org/wiki/xacro">
     <!-- Center of buoyancy -->
-    <xacro:property name="maelstrom_cob" value="0.0205 0 0.04"/>
+    <xacro:property name="maelstrom_cob" value="0 0 0"/>
     <!-- Vehicle's actual volume (Gazebo cannot compute the volume out of the mesh) -->
     <xacro:property name="maelstrom_volume" value="0.0386"/>
@@ -25,25 +25,18 @@
     <xacro:property name="maelstrom_hydro_model">
         <type>fossen</type>
-        <!-- Added mass: see p.28 in Berg2012 -->
         <added_mass>
-            0 0 0 0 0 0
-            0 82.4183 0 0 0 26.2914
-            0 0 82.4183 0 26.2914 0
-            0 0 0 0 0 0
-            0 0 26.2914 0 11.1826 0
-            0 26.1914 0 0 0 11.1826
+        1.7 0 0 0 0 0
+        0 0 0 0 0 0
+        0 0 5 0 0 0
+        0 0 0 0 0 0
+        0 0 0 1.5 0 0
+        0 0 0 0 0 .4
         </added_mass>
-        <!-- Linear damping: see p.31 in Berg2012 -->
         <linear_damping>
-            -74.82 -69.48 -728.4 -268.8 -309.77 -105
+        -11.7391 -20 -31.8678 -25 -44.9085 -5
         </linear_damping>
-        <!-- Non-linear damping: see p.30 in Berg2012 -->
-        <quadratic_damping>
-            -748.22 -992.53 -1821.01 -672 -774.44 -523.27
-        </quadratic_damping>
     </xacro:property>
-    <xacro:property name="max_thrust" value="10" />
-    <xacro:property name="min_thrust" value="-10" />
-    <!--TODO: Rotate mesh aswell -->
+    <xacro:property name="max_thrust" value="24" />
+    <xacro:property name="min_thrust" value="-24" />
     <xacro:property name="hpf_pos"><origin xyz="0.37273 0.18946 -0.01509" rpy="0 ${pi/2} 0" /></xacro:property>
     <xacro:property name="hpa_pos"><origin xyz="-0.32577 0.18946 -0.01509" rpy="0 ${pi/2} 0" /></xacro:property>

File: maelstrom_description/urdf/snippets.xacro (robot description, xacro)
@@ -86,5 +86,5 @@
         <conversion>
           <type>Basic</type>
-          <rotorConstant>0.00031</rotorConstant>
+          <rotorConstant>0.005</rotorConstant>
         </conversion>
       </plugin>

Commit message: single launch file added: simulation.launch

File: maelstrom_description/urdf/properties.xacro (robot description, xacro)
@@ -2,7 +2,7 @@
 <robot xmlns:xacro="http://www.ros.org/wiki/xacro">
     <!-- Center of buoyancy -->
-    <xacro:property name="maelstrom_cob" value="0 0 0"/>
+    <xacro:property name="maelstrom_cob" value=".027 -.002 .08"/>
     <!-- Vehicle's actual volume (Gazebo cannot compute the volume out of the mesh) -->
-    <xacro:property name="maelstrom_volume" value="0.0386"/>
+    <xacro:property name="maelstrom_volume" value="0.0428"/>
     <!-- Describing the dimensions of the vehicle's bounding box -->
     <xacro:property name="maelstrom_length" value="0.782"/>
@@ -11,5 +11,5 @@
       <!-- Fluid density -->
      <xacro:property name="rho" value="1028" />
-    <xacro:property name="maelstrom_mass" value="36.1"/>
+    <xacro:property name="maelstrom_mass" value="40.85"/>
     <!-- Center of gravity -->
     <xacro:property name="maelstrom_cog" value="0 0 0"/>

Commit message: DVL plugin, make properties 0

File: maelstrom_description/urdf/properties.xacro (robot description, xacro)
@@ -2,5 +2,5 @@
 <robot xmlns:xacro="http://www.ros.org/wiki/xacro">
     <!-- Center of buoyancy -->
-    <xacro:property name="maelstrom_cob" value=".027 -.002 .08"/>
+    <xacro:property name="maelstrom_cob" value="0 0 0"/>
     <!-- Vehicle's actual volume (Gazebo cannot compute the volume out of the mesh) -->
     <xacro:property name="maelstrom_volume" value="0.0428"/>
@@ -18,7 +18,7 @@
             <mass value="${maelstrom_mass}" />
             <origin xyz="${maelstrom_cog}" rpy="0 0 0"/>
-            <inertia ixx="0.69" ixy="0" ixz="0"
-                    iyy="2.62" iyz="0"
-                    izz="2.51" />
+            <inertia ixx="0" ixy="0" ixz="0"
+                    iyy="0" iyz="0"
+                    izz="0" />
         </inertial>
     </xacro:property>
@@ -26,10 +26,10 @@
         <type>fossen</type>
         <added_mass>
-        1.7 0 0 0 0 0
         0 0 0 0 0 0
-        0 0 5 0 0 0
         0 0 0 0 0 0
-        0 0 0 1.5 0 0
-        0 0 0 0 0 .4
+        0 0 0 0 0 0
+        0 0 0 0 0 0
+        0 0 0 0 0 0
+        0 0 0 0 0 0
         </added_mass>
         <linear_damping>
