Commit message: Fixed .so errors

File: maelstrom_description/robots/default.xacro (robot description, xacro)
@@ -12,5 +12,5 @@
      allow the addition of external models of manipulator units -->
     <gazebo>
-      <plugin name="uuv_plugin" filename="libunderwater_object_ros_plugin.so">
+      <plugin name="uuv_plugin" filename="libuuv_underwater_object_ros_plugin.so">
         <fluid_density>1028.0</fluid_density>
         <flow_velocity_topic>hydrodynamics/current_velocity</flow_velocity_topic>

File: maelstrom_description/urdf/properties.xacro (robot description, xacro)
@@ -18,7 +18,7 @@
             <mass value="${maelstrom_mass}" />
             <origin xyz="${maelstrom_cog}" rpy="0 0 0"/>
-            <inertia ixx="0" ixy="0" ixz="0"
-                    iyy="0" iyz="0"
-                    izz="0" />
+            <inertia ixx="1.32" ixy="0" ixz="0"
+                    iyy="2.84" iyz="0"
+                    izz="3.65" />
         </inertial>
     </xacro:property>

File: maelstrom_description/urdf/snippets.xacro (robot description, xacro)
@@ -37,5 +37,5 @@
     <gazebo>
       <!-- Thruster ROS plugin -->
-      <plugin name="${robot_namespace}_${thruster_id}_thruster_model" filename="libthruster_ros_plugin.so">
+      <plugin name="${robot_namespace}_${thruster_id}_thruster_model" filename="libuuv_thruster_ros_plugin.so">
         <!-- Name of the thruster link -->
         <linkName>${robot_namespace}/thruster_${thruster_id}</linkName>

Commit message: Renamed cfgs, added depth pub

File: maelstrom_description/robots/default.xacro (robot description, xacro)
@@ -13,5 +13,5 @@
     <gazebo>
       <plugin name="uuv_plugin" filename="libuuv_underwater_object_ros_plugin.so">
-        <fluid_density>1028.0</fluid_density>
+        <fluid_density>1000.0</fluid_density>
         <flow_velocity_topic>hydrodynamics/current_velocity</flow_velocity_topic>
         <debug>$(arg debug)</debug>

File: maelstrom_description/urdf/properties.xacro (robot description, xacro)
@@ -10,5 +10,5 @@
     <xacro:property name="maelstrom_height" value="0.967"/>
       <!-- Fluid density -->
-     <xacro:property name="rho" value="1028" />
+     <xacro:property name="rho" value="1000" />
     <xacro:property name="maelstrom_mass" value="40.85"/>
     <!-- Center of gravity -->
@@ -37,6 +37,6 @@
         </linear_damping>
     </xacro:property>
-    <xacro:property name="max_thrust" value="24" />
-    <xacro:property name="min_thrust" value="-24" />
+    <xacro:property name="max_thrust" value="40" />
+    <xacro:property name="min_thrust" value="-40" />
     <xacro:property name="hpf_pos"><origin xyz="0.37273 0.18946 -0.01509" rpy="0 ${pi/2} 0" /></xacro:property>
     <xacro:property name="hpa_pos"><origin xyz="-0.32577 0.18946 -0.01509" rpy="0 ${pi/2} 0" /></xacro:property>
