Commit message: Added common robot description, changing maelstrom xacro files

File: maelstrom_description/model/robots/maelstrom.urdf.xacro (robot description, xacro)
@@ -4,7 +4,8 @@
   <xacro:arg name="namespace" default="maelstrom"/>
   <!-- Include the ROV macro file -->
-  <xacro:include filename="$(find maelstrom_description)/urdf/properties.xacro" />
-  <xacro:include filename="$(find maelstrom_description)/urdf/base.xacro"/>
-  <xacro:include filename="$(find maelstrom_description)/urdf/gazebo.xacro"/>
+  <xacro:include filename="$(find maelstrom_description)/model/xacro/base.xacro" />
+  <xacro:include filename="$(find maelstrom_description)/model/xacro/thrusters.xacro"/>
+  <xacro:include filename="$(find maelstrom_description)/model/xacro/sensors.xacro"/>
+  <xacro:include filename="$(find maelstrom_description)/model/xacro/gazebo.xacro"/>
   <!-- Create the maelstrom -->
   <xacro:maelstrom_base namespace="$(arg namespace)">

File: maelstrom_description/model/xacro/base.xacro (robot description, xacro)
@@ -31,5 +31,5 @@
     <joint name="inert_base" type="fixed">
       <parent link="${namespace}/base_link"/>
-      <child link="${namespace}/inert"/>
+      <child link="${namespace}/inertia"/>
     </joint>
     <gazebo reference="${namespace}/base_link">

File: maelstrom_description/model/xacro/snippets.xacro (robot description, xacro)
@@ -32,5 +32,5 @@
       <xacro:insert_block name="origin" />
       <axis xyz="1 0 0" />
-      <parent link="${robot_namespace}/inert" />
+      <parent link="${robot_namespace}/inertia" />
       <child link="${robot_namespace}/thruster_${thruster_id}" />
     </joint>
