Commit message: Wrote thrust converter. Still have to test

File: common_robot_description/xacro/common_thrusters.xacro (robot description, xacro)
@@ -26,5 +26,5 @@
         <linkName>${data[tag_link][tag_name]}</linkName>
         <jointName>${data[tag_joint][tag_name]}</jointName>
-        <thrusterID>${data[tag_thruster][tag_id]}</thrusterID>
+        <thrusterID>${data[tag_id]}</thrusterID>
         <thrustMax>${t200[tag_limits][tag_thrust][tag_max]}</thrustMax>
         <thrustMin>${t200[tag_limits][tag_thrust][tag_min]}</thrustMin>
@@ -47,3 +47,36 @@
     </gazebo>
   </xacro:macro>
+  <xacro:macro name="uuv_thruster_from_yaml" params="data">
+    <!--
+    Dummy link as place holder for the thruster frame,
+    since thrusters can often be inside the collision geometry
+    of the vehicle and may cause internal collisions if set otherwise
+    -->
+    <xacro:standard_link_from_yaml data="${data[tag_link][tag_name]}"/>
+    <xacro:standard_joint_from_yaml data="${data[tag_joint]}" child="${data[tag_link][tag_name]}"/>
+    <gazebo>
+      <plugin name="${data[tag_link][tag_name]}_model" filename="libuuv_thruster_ros_plugin.so">
+        <linkName>${data[tag_link][tag_name]}</linkName>
+        <jointName>${data[tag_joint][tag_name]}</jointName>
+        <thrusterID>${data[tag_id]}</thrusterID>
+        <thrustMax>${data[tag_limits][tag_thrust][tag_max]}</thrustMax>
+        <thrustMin>${data[tag_limits][tag_thrust][tag_min]}</thrustMin>
+        <dynamics>
+          <type>${data[tag_gazebo][tag_dynamics]}</type>
+        </dynamics>
+        <!-- Basic curve
+        Input: x
+        Output: thrust
+        Function: thrust = rotorConstant * x * abs(x)
+        -->
+        <conversion>
+          <type>${data[tag_gazebo][tag_conversion][tag_type]}</type>
+          <rotorConstant>${data[tag_gazebo][tag_conversion][tag_constant]}</rotorConstant>
+        </conversion>
+      </plugin>
+    </gazebo>
+    <gazebo reference="${data[tag_link][tag_name]}">
+      <selfCollide>false</selfCollide>
+    </gazebo>
+  </xacro:macro>
 </robot>

File: maelstrom_description/model/xacro/sensors.xacro (robot description, xacro)
@@ -8,6 +8,7 @@
    <xacro:camera_from_yaml data="${sensors_data['camera']['forward_L']}"/>
    <xacro:camera_from_yaml data="${sensors_data['camera']['downward']}"/>
+   <!-- Only an IMU is needed among the inertial sensors, but all are included to represent the actual vehicle -->
+   <xacro:imu_from_yaml data="${sensors_data['imu']['imu']}"/>
    <xacro:pressure_from_yaml data="${sensors_data['pressure']['pressure']}"/>
-   <xacro:imu_from_yaml data="${sensors_data['imu']['imu']}"/>
    <xacro:dvl_from_yaml data="${sensors_data['dvl']['dvl']}"/>
 </robot>

Commit message: Simulator in full working condition

File: common_robot_description/xacro/common_thrusters.xacro (robot description, xacro)
@@ -11,7 +11,7 @@
   <xacro:property name="tag_dynamics" value="dynamics"/>
   <!-- Load Blue Robotics T200 Data -->
-  <xacro:property name="t200_file" value="$(find common_robot_description)/config/thruster_t200.yaml"/>
-  <xacro:property name="t200_data" value="${load_yaml(t200_file)}"/>
-  <xacro:property name="t200" value="${t200_data['t200']}"/>
+  <xacro:property name="common_thrusters_file" value="$(find common_robot_description)/config/common_thrusters.yaml"/>
+  <xacro:property name="common_thrusters_data" value="${load_yaml(common_thrusters_file)}"/>
+  <xacro:property name="T200" value="${common_thrusters_data['T200']}"/>
   <xacro:macro name="uuv_thruster_t200_from_yaml" params="data">
     <!--
@@ -20,5 +20,5 @@
     of the vehicle and may cause internal collisions if set otherwise
     -->
-    <xacro:standard_link_from_yaml name="${data[tag_link][tag_name]}" data="${t200[tag_link]}"/>
+    <xacro:standard_link_from_yaml name="${data[tag_link][tag_name]}" data="${T200[tag_link]}"/>
     <xacro:standard_joint_from_yaml data="${data[tag_joint]}" child="${data[tag_link][tag_name]}"/>
     <gazebo>
@@ -27,8 +27,8 @@
         <jointName>${data[tag_joint][tag_name]}</jointName>
         <thrusterID>${data[tag_id]}</thrusterID>
-        <thrustMax>${t200[tag_limits][tag_thrust][tag_max]}</thrustMax>
-        <thrustMin>${t200[tag_limits][tag_thrust][tag_min]}</thrustMin>
+        <thrustMax>${T200[tag_limits][tag_thrust][tag_max]}</thrustMax>
+        <thrustMin>${T200[tag_limits][tag_thrust][tag_min]}</thrustMin>
         <dynamics>
-          <type>${t200[tag_gazebo][tag_dynamics]}</type>
+          <type>${T200[tag_gazebo][tag_dynamics]}</type>
         </dynamics>
         <!-- Basic curve
@@ -38,6 +38,6 @@
         -->
         <conversion>
-          <type>${t200[tag_gazebo][tag_conversion][tag_type]}</type>
-          <rotorConstant>${t200[tag_gazebo][tag_conversion][tag_constant]}</rotorConstant>
+          <type>${T200[tag_gazebo][tag_conversion][tag_type]}</type>
+          <rotorConstant>${T200[tag_gazebo][tag_conversion][tag_constant]}</rotorConstant>
         </conversion>
       </plugin>
