Commit message: Tried reworking xacro files.

File: common_robot_description/xacro/common_joints.xacro (robot description, xacro)
@@ -2,5 +2,9 @@
 <robot xmlns:xacro="http://www.ros.org/wiki/xacro" name="common_links">
   <xacro:include filename="$(find common_robot_description)/xacro/common_tags.xacro"/>
-  <xacro::macro name="standard_joint_from_yaml" params="name:=None data child">
+  <xacro:property name="tag_axis" value="axis"/>
+  <xacro:property name="tag_damping" value="damping"/>
+  <xacro:property name="tag_dynamics" value="dynamics"/>
+  <xacro:property name="tag_parent" value="parent"/>
+  <xacro:macro name="standard_joint_from_yaml" params="name:=None data child">
    <joint name="${data[tag_name] if name is None else name}" type="${data[tag_type]}">
       <origin xyz="${data[tag_origin][tag_xyz]}"

File: common_robot_description/xacro/common_links.xacro (robot description, xacro)
@@ -2,9 +2,78 @@
 <robot xmlns:xacro="http://www.ros.org/wiki/xacro" name="common_links">
   <xacro:include filename="$(find common_robot_description)/xacro/common_tags.xacro"/>
-  <xacro::macro name="inertia_from_yaml" params="data">
+  <!-- Link Tags -->
+  <xacro:property name="tag_collision" value="collision"/>
+  <xacro:property name="tag_com" value="com"/>
+  <xacro:property name="tag_dummy_joint" value="dummy_joint"/>
+  <xacro:property name="tag_dummy_link" value="dummy_link"/>
+  <xacro:property name="tag_inertia" value="inertia"/>
+  <xacro:property name="tag_ixx" value="ixx"/>
+  <xacro:property name="tag_ixy" value="ixy"/>
+  <xacro:property name="tag_ixz" value="ixz"/>
+  <xacro:property name="tag_iyy" value="iyy"/>
+  <xacro:property name="tag_iyz" value="iyz"/>
+  <xacro:property name="tag_izz" value="izz"/>
+  <xacro:property name="tag_mass" value="mass"/>
+  <xacro:property name="tag_mesh" value="mesh_properties"/>
+  <xacro:property name="tag_visual" value="visual"/>
+  <!-- Hydro Link Tags -->
+  <xacro:property name="tag_added_mass" value="added_mass"/>
+  <xacro:property name="tag_box" value="box"/>
+  <xacro:property name="tag_constant" value="constant"/>
+  <xacro:property name="tag_cob" value="cob"/>
+  <xacro:property name="tag_damping" value="damping"/>
+  <xacro:property name="tag_height" value="height"/>
+  <xacro:property name="tag_hydro" value="hydro"/>
+  <xacro:property name="tag_length" value="length"/>
+  <xacro:property name="tag_linear" value="linear"/>
+  <xacro:property name="tag_quadratic" value="quadratic"/>
+  <xacro:property name="tag_volume" value="volume"/>
+  <xacro:property name="tag_width" value="width"/>
+  <xacro:macro name="inertia_from_yaml" params="data">
     <inertia ixx="${data[tag_ixx]}" ixy="${data[tag_ixy]}" ixz="${data[tag_ixz]}"
              iyy="${data[tag_iyy]}" iyz="${data[tag_iyz]}" izz="${data[tag_izz]}"/>
   </xacro:macro>
-  <xacro::macro name="standard_link_from_yaml" params="name:=None data">
+  <xacro:macro name="base_link_from_yaml" params="data">
+    <link name="${data[tag_name]}">
+      <xacro:if value="${tag_mesh in data}">
+        <xacro:if value="${tag_visual in data[tag_mesh]}">
+          <visual>
+            <geometry>
+              <mesh filename="${data[tag_mesh][tag_visual]}" scale="1 1 1"/>
+            </geometry>
+            <origin xyz="0.0 0.0 0.0" rpy="0.0 0.0 0.0"/>
+          </visual>
+        </xacro:if>
+        <xacro:if value="${tag_collision in data[tag_mesh]}">
+          <visual>
+            <geometry>
+              <mesh filename="${data[tag_mesh][tag_collision]}" scale="1 1 1"/>
+            </geometry>
+            <origin xyz="0.0 0.0 0.0" rpy="0.0 0.0 0.0"/>
+          </visual>
+        </xacro:if>
+      </xacro:if>
+    </link>
+    <link name="${data[tag_dummy_link][tag_name]}">
+      <inertial>
+        <mass value="${data[tag_mass]}"/>
+        <origin xyz="${data[tag_com][tag_x]} ${data[tag_com][tag_y]} ${data[tag_com][tag_z]}" rpy="0 0 0"/>
+        <inertia ixx="${data[tag_inertia][tag_ixx]}"
+                ixy="${data[tag_inertia][tag_ixy]}"
+                ixz="${data[tag_inertia][tag_ixz]}"
+                iyy="${data[tag_inertia][tag_iyy]}"
+                iyz="${data[tag_inertia][tag_iyz]}"
+                izz="${data[tag_inertia][tag_izz]}" />
+      </inertial>
+    </link>
+    <joint name="${data[tag_dummy_joint][tag_name]}" type="fixed">
+      <parent link="${data[tag_name]}"/>
+      <child link="${data[tag_dummy_link][tag_name]}"/>
+    </joint>
+    <gazebo reference="${data[tag_name]}">
+      <selfCollide>false</selfCollide>
+    </gazebo>
+  </xacro:macro>
+  <xacro:macro name="standard_link_from_yaml" params="name:=None data">
     <link name="${data[tag_name] if name is None else name}">
       <xacro:if value="${tag_mesh in data}">
@@ -17,5 +86,5 @@
           </visual>
         </xacro:if>
-        <xacro:if value="${tag_collision in data[tag_link][tag_mesh]}">
+        <xacro:if value="${tag_collision in data[tag_mesh]}">
           <visual>
             <geometry>
@@ -38,5 +107,5 @@
     </link>
   </xacro:macro>
-  <xacro:macro name="uuv_hydro_link_from_yaml" params="name data">
+  <xacro:macro name="hydro_link_from_yaml" params="name data">
     <link name="${name}">
       <volume>${data[tag_volume]}</volume>
@@ -51,5 +120,5 @@
         </box>
       </xacro:if>
-      <center_of_buoyancy>${data[tag_cob]}</center_of_buoyancy>
+      <center_of_buoyancy>${data[tag_cob]}</center_of_buoyancy> <!-- In the body frame -->
       <hydrodynamic_model>
         <type>fossen</type>
@@ -60,3 +129,12 @@
     </link>
   </xacro:macro>
+  <xacro:macro name="uuv_hydro_links" params="flow_topic:='hydrodynamics/current_velocity' fluid_density:=1000 **uuv_links">
+    <gazebo>
+      <plugin name="uuv_plugin" filename="libuuv_underwater_object_ros_plugin.so">
+        <fluid_density>${fluid_density}</fluid_density>
+        <flow_velocity_topic>${flow_topic}</flow_velocity_topic>
+        <xacro:insert_block name="uuv_links"/>
+      </plugin>
+    </gazebo>
+  </xacro:macro>
 </robot>

File: common_robot_description/xacro/common_tags.xacro (robot description, xacro)
@@ -1,43 +1,20 @@
 <?xml version="1.0"?>
 <robot xmlns:xacro="http://www.ros.org/wiki/xacro" name="common_tags">
-  <xacro:property name="tag_gazebo" value="gazebo">
-  <xacro:property name="tag_id" value="id">
-  <xacro:property name="tag_joint" value="joint">
-  <xacro:property name="tag_link" value="link">
-  <xacro:property name="tag_limits" value="limits">
-  <xacro:property name="tag_max" value="max">
-  <xacro:property name="tag_min" value="min">
-  <xacro:property name="tag_model" value="model">
-  <xacro:property name="tag_name" value="name">
-  <xacro:property name="tag_origin" value="origin">
-  <xacro:property name="tag_rpy" value="rpy">
-  <xacro:property name="tag_thrust" value="thrust">
-  <xacro:property name="tag_thruster" value="thruster">
-  <xacro:property name="tag_type" value="type">
-  <xacro:property name="tag_added_mass" value="added_mass">
-  <xacro:property name="tag_box" value="box">
-  <xacro:property name="tag_constant" value="constant">
-  <xacro:property name="tag_cob" value="cob">
-  <xacro:property name="tag_collision" value="collision">
-  <xacro:property name="tag_com" value="com">
-  <xacro:property name="tag_conversion" value="thruster_conversion">
-  <xacro:property name="tag_damping" value="damping">
-  <xacro:property name="tag_dynamics" value="dynamics">
-  <xacro:property name="tag_hydro" value="hydro">
-  <xacro:property name="tag_inertia" value="inertia">
-  <xacro:property name="tag_ixx" value="ixx">
-  <xacro:property name="tag_ixy" value="ixy">
-  <xacro:property name="tag_ixz" value="ixz">
-  <xacro:property name="tag_iyy" value="iyy">
-  <xacro:property name="tag_iyz" value="iyz">
-  <xacro:property name="tag_izz" value="izz">
-  <xacro:property name="tag_linear" value="linear">
-  <xacro:property name="tag_mass" value="mass">
-  <xacro:property name="tag_mesh" value="mesh_properties">
-  <xacro:property name="tag_quadratic" value="quadratic">
-  <xacro:property name="tag_visual" value="visual">
-  <xacro:property name="tag_volume" value="volume">
-  <xacro:property name="tag_x" value="x">
-  <xacro:property name="tag_y" value="y">
-  <xacro:property name="tag_z" value="z">
+  <!-- Shared Tags -->
+  <xacro:property name="tag_gazebo" value="gazebo"/>
+  <xacro:property name="tag_id" value="id"/>
+  <xacro:property name="tag_joint" value="joint"/>
+  <xacro:property name="tag_limits" value="limits"/>
+  <xacro:property name="tag_link" value="link"/>
+  <xacro:property name="tag_max" value="max"/>
+  <xacro:property name="tag_min" value="min"/>
+  <xacro:property name="tag_name" value="name"/>
+  <xacro:property name="tag_origin" value="origin"/>
+  <xacro:property name="tag_plugin" value="plugin"/>
+  <xacro:property name="tag_rpy" value="rpy"/>
+  <xacro:property name="tag_type" value="type"/>
+  <xacro:property name="tag_x" value="x"/>
+  <xacro:property name="tag_xyz" value="xyz"/>
+  <xacro:property name="tag_y" value="y"/>
+  <xacro:property name="tag_z" value="z"/>
 </robot>

File: common_robot_description/xacro/common_thrusters.xacro (robot description, xacro)
@@ -4,7 +4,14 @@
   <xacro:include filename="$(find common_robot_description)/xacro/common_links.xacro"/>
   <xacro:include filename="$(find common_robot_description)/xacro/common_joints.xacro"/>
+  <!-- Thruster Tags -->
+  <xacro:property name="tag_thrust" value="thrust"/>
+  <xacro:property name="tag_thruster" value="thruster"/>
+  <xacro:property name="tag_conversion" value="thrust_conversion"/>
+  <xacro:property name="tag_dynamics" value="dynamics"/>
+  <!-- Load Blue Robotics T200 Data -->
   <xacro:property name="t200_file" value="$(find common_robot_description)/config/thruster_t200.yaml"/>
   <xacro:property name="t200_data" value="${load_yaml(t200_file)}"/>
-  <xacro:macro name="thruster_t200_from_yaml" params="data">
+  <xacro:property name="t200" value="${t200_data['t200']}"/>
+  <xacro:macro name="uuv_thruster_t200_from_yaml" params="data">
     <!--
     Dummy link as place holder for the thruster frame,
@@ -12,5 +19,5 @@
     of the vehicle and may cause internal collisions if set otherwise
     -->
-    <xacro:standard_link_from_yaml name="${data[tag_link][tag_name]}" data="${t200_data[tag_link]}"/>
+    <xacro:standard_link_from_yaml name="${data[tag_link][tag_name]}" data="${t200[tag_link]}"/>
     <xacro:standard_joint_from_yaml data="${data[tag_joint]}" child="${data[tag_link][tag_name]}"/>
     <!--<link name="${data[tag_link][tag_name]}">
@@ -46,8 +53,8 @@
         <thrusterID>${data[tag_thruster][tag_id]}</thrusterID>
         <!-- Minimum and maximum thrust force output allowed -->
-        <thrustMax>${t200_data[tag_limits][tag_thrust][tag_max]}</thrustMax>
-        <thrustMin>${t200_data[tag_limits][tag_thrust][tag_min]}</thrustMin>
+        <thrustMax>${t200[tag_limits][tag_thrust][tag_max]}</thrustMax>
+        <thrustMin>${t200[tag_limits][tag_thrust][tag_min]}</thrustMin>
         <dynamics>
-          <type>${t200_data[tag_gazebo][tag_dynamics]}</type>
+          <type>${t200[tag_gazebo][tag_dynamics]}</type>
         </dynamics>
         <!-- Basic curve
@@ -58,6 +65,6 @@
         <!-- TODO: Find good thruster model -->
         <conversion>
-          <type>${t200_data[tag_gazebo][tag_conversion][tag_type]}</type>
-          <rotorConstant>${t200_data[tag_gazebo][tag_conversion][tag_constant]}</rotorConstant>
+          <type>${t200[tag_gazebo][tag_conversion][tag_type]}</type>
+          <rotorConstant>${t200[tag_gazebo][tag_conversion][tag_constant]}</rotorConstant>
         </conversion>
       </plugin>

File: maelstrom_description/model/robots/maelstrom.urdf.xacro (robot description, xacro)
@@ -3,30 +3,21 @@
   <xacro:arg name="debug" default="0"/>
   <xacro:arg name="namespace" default="maelstrom"/>
-  <!-- Include the ROV macro file -->
-  <xacro:include filename="$(find maelstrom_description)/model/xacro/base.xacro" />
+  <xacro:property name="namespace" value="$(arg namespace)"/>
+  <!-- Include common xacros -->
+  <xacro:include filename="$(find uuv_descriptions)/urdf/common.urdf.xacro"/>
+  <xacro:include filename="$(find common_robot_description)/xacro/common_tags.xacro"/>
+  <xacro:include filename="$(find common_robot_description)/xacro/common_links.xacro"/>
+  <xacro:include filename="$(find common_robot_description)/xacro/common_joints.xacro"/>
+  <!-- Create Maelstrom -->
+  <xacro:include filename="$(find maelstrom_description)/model/xacro/base.xacro"/>
   <xacro:include filename="$(find maelstrom_description)/model/xacro/thrusters.xacro"/>
   <xacro:include filename="$(find maelstrom_description)/model/xacro/sensors.xacro"/>
-  <xacro:include filename="$(find maelstrom_description)/model/xacro/gazebo.xacro"/>
-  <!-- Create the maelstrom -->
-  <xacro:maelstrom_base namespace="$(arg namespace)">
-    <!-- The underwater object plugin is given as an input block parameter to
-     allow the addition of external models of manipulator units -->
-    <gazebo>
-      <plugin name="uuv_plugin" filename="libuuv_underwater_object_ros_plugin.so">
-        <fluid_density>1000.0</fluid_density>
-        <flow_velocity_topic>hydrodynamics/current_velocity</flow_velocity_topic>
-        <debug>$(arg debug)</debug>
-        <!-- Adding the hydrodynamic and hydrostatic parameters for the vehicle-->
-        <xacro:maelstrom_hydro_model namespace="$(arg namespace)"/>
-        <!--
-          In case other modules are added to the vehicle (such as a manipulator)
-          that also have link running with the underwater object plugin, they
-          should also be added in this block. For this, this new module should
-          have a file similar to gazebo.xacro above with the description of the
-          parameter necessary for the underwater object plugin to be initialized.
-        -->
-      </plugin>
-    </gazebo>
-  </xacro:maelstrom_base>
+  <!-- Combine hydro links -->
+  <!-- Can add more within uuv_links as the model grows -->
+  <xacro:uuv_hydro_links>
+    <uuv_links>
+      <xacro:maelstrom_base_uuv_links/>
+    </uuv_links>
+  </xacro:uuv_hydro_links>
   <!-- Joint state publisher plugin -->
   <xacro:default_joint_state_publisher namespace="$(arg namespace)" update_rate="10"/>

File: maelstrom_description/model/xacro/base.xacro (robot description, xacro)
@@ -1,45 +1,13 @@
 <?xml version="1.0"?>
-<robot xmlns:xacro="http://www.ros.org/wiki/xacro">
-  <!-- Loading some constants -->
-  <xacro:include filename="$(find uuv_descriptions)/urdf/common.urdf.xacro"/>
-  <!-- Loading file with sensor macros -->
-  <xacro:include filename="$(find uuv_sensor_ros_plugins)/urdf/sensor_snippets.xacro"/>
-  <!-- Loading the UUV simulator ROS plugin macros -->
-  <xacro:include filename="$(find uuv_gazebo_ros_plugins)/urdf/snippets.xacro"/>
-  <!-- Loading vehicle's specific macros -->
-  <xacro:include filename="$(find maelstrom_description)/urdf/snippets.xacro"/>
-  <!-- Vehicle macro -->
-  <xacro:macro name="maelstrom_base" params="namespace *gazebo">
-      <!-- Rigid body description of the base link -->
-      <link name="${namespace}/base_link">
-        <visual>
-          <origin xyz="0 0 0" rpy="0 0 0"/>
-          <geometry>
-            <mesh filename="${visual_mesh_file}" scale="1 1 1" />
-          </geometry>
-        </visual>
-        <collision>
-          <origin xyz="0 0 0" rpy="0 0 0"/>
-          <geometry>
-            <mesh filename="${collision_mesh_file}" scale="1 1 1" />
-          </geometry>
-        </collision>
-      </link>
-      <link name="${namespace}/inert">
-        <xacro:insert_block name="maelstrom_inertia" />
-      </link>
-    <joint name="inert_base" type="fixed">
-      <parent link="${namespace}/base_link"/>
-      <child link="${namespace}/inertia"/>
-    </joint>
-    <gazebo reference="${namespace}/base_link">
-      <selfCollide>false</selfCollide>
-    </gazebo>
-    <!-- Set up hydrodynamic plugin given as input parameter -->
-    <xacro:insert_block name="gazebo"/>
-    <!-- Include the thruster modules -->
-    <xacro:include filename="$(find maelstrom_description)/urdf/actuators.xacro"/>
-    <!-- Include the sensor modules -->
-    <xacro:include filename="$(find maelstrom_description)/urdf/sensors.xacro"/>
+<robot xmlns:xacro="http://www.ros.org/wiki/xacro" name="base">
+  <xacro:include filename="$(find common_robot_description)/xacro/common_tags.xacro"/>
+  <xacro:include filename="$(find common_robot_description)/xacro/common_links.xacro"/>
+  <!-- Load Maelstrom Base Data -->
+  <xacro:property name="base_file" value="$(find maelstrom_description)/model/config/base.yaml"/>
+  <xacro:property name="base_data" value="${load_yaml(base_file)}"/>
+  <xacro:property name="base" value="${base_data['base_link']}"/>
+  <xacro:base_link_from_yaml data="${base[tag_link]}"/>
+  <xacro:macro name="maelstrom_base_uuv_links">
+    <xacro:hydro_link_from_yaml name="${base[tag_link][tag_name]}" data="${base[tag_link][tag_hydro]}"/>
   </xacro:macro>
 </robot>

File: maelstrom_description/model/xacro/sensors.xacro (robot description, xacro)
@@ -2,4 +2,7 @@
 <robot xmlns:xacro="http://www.ros.org/wiki/xacro">
 	<xacro:include filename="$(find uuv_sensor_ros_plugins)/urdf/sensor_snippets.xacro"/>
+	<xacro:property name="forward_camera_R_pos"><origin xyz="0.3818 0.05038 0.11999" rpy="0 0 0" /></xacro:property>
+    <xacro:property name="forward_camera_L_pos"><origin xyz="0.3818 -0.05038 0.11999" rpy="0 0 0" /></xacro:property>
+    <xacro:property name="downward_camera_pos"><origin xyz="0.0711 0.0004 0" rpy="0 ${pi/2} 0" /></xacro:property>
   <!--
     Some examples of sensors that can be added to the vehicle frame.
@@ -12,5 +15,5 @@
 				namespace="sensors"
 				suffix="_forward_R"
-				parent_link="${namespace}/base_link"
+				parent_link="base_link"
 				topic="camera"
 				mass="0.001"
@@ -28,5 +31,5 @@
 				namespace="sensors"
 				suffix="_forward_L"
-				parent_link="${namespace}/base_link"
+				parent_link="base_link"
 				topic="camera"
 				mass="0.001"
@@ -44,5 +47,5 @@
 				namespace="sensors"
 				suffix="_downward"
-				parent_link="${namespace}/base_link"
+				parent_link="base_link"
 				topic="camera"
 				mass="0.001"
@@ -59,5 +62,5 @@
 	<xacro:default_imu_macro
 				namespace="${namespace}"
-				parent_link="${namespace}/base_link"
+				parent_link="base_link"
 				inertial_reference_frame="world_ned">
 				<origin xyz="0 0 0" rpy="0 0 0"/>
@@ -66,10 +69,10 @@
 	<xacro:default_dvl_macro
 				namespace="${namespace}"
-				parent_link="${namespace}/base_link"
+				parent_link="base_link"
 				inertial_reference_frame="world_ned">
 				<origin xyz="-0.081297 -0.081297 0.0" rpy="0 ${0.5*pi} 0"/>
 	</xacro:default_dvl_macro>
 	<!--Depth Sensor-->
-	<xacro:default_pressure_macro namespace="${namespace}" parent_link="${namespace}/base_link">
+	<xacro:default_pressure_macro namespace="${namespace}" parent_link="base_link">
 				<origin xyz="0 -0.0004 0.0711" rpy="0 0 0"/>
 	</xacro:default_pressure_macro>

File: maelstrom_description/model/xacro/thrusters.xacro (robot description, xacro)
@@ -1,22 +1,18 @@
 <?xml version="1.0"?>
-<robot xmlns:xacro="http://www.ros.org/wiki/xacro">
-    <!-- Adding the thruster units with the macro created in snippets.xacro -->
-    <!--
-    Important:
-        - The thruster IDs must be given as integers and must be unique to each thruster unit
-        - The thruster pose in the <origin> block is relative to the body's center of mass. Be
-          aware that Gazebo does not use the SNAME convention per default.
-    -->
+<robot xmlns:xacro="http://www.ros.org/wiki/xacro" name="thrusters">
+    <!-- Include needed xacros -->
+    <xacro:include filename="$(find uuv_gazebo_ros_plugins)/urdf/snippets.xacro"/>
     <xacro:include filename="$(find common_robot_description)/xacro/common_thrusters.xacro"/>
-    <xacro:include filename="$(find maelstrom_description)/model/xacro/thrusters.xacro"/>
+    <!-- Load data from yaml -->
     <xacro:property name="thruster_file" value="$(find maelstrom_description)/model/config/thrusters.yaml"/>
     <xacro:property name="thruster_data" value="${load_yaml(thruster_file)}"/>
-    <xacro:thruster_t200_from_yaml name="thruster_hpf" value="${thruster_data['heave_port_fwd])}"/>
-    <xacro:thruster_t200_from_yaml name="thruster_hpa" value="${thruster_data['heave_port_aft])}"/>
-    <xacro:thruster_t200_from_yaml name="thruster_hsf" value="${thruster_data['heave_stbd_fwd])}"/>
-    <xacro:thruster_t200_from_yaml name="thruster_hsa" value="${thruster_data['heave_stbd_aft])}"/>
-    <xacro:thruster_t200_from_yaml name="thruster_vpf" value="${thruster_data['vector_port_fwd])}"/>
-    <xacro:thruster_t200_from_yaml name="thruster_vpa" value="${thruster_data['vector_port_aft])}"/>
-    <xacro:thruster_t200_from_yaml name="thruster_vsf" value="${thruster_data['vector_stbd_fwd])}"/>
-    <xacro:thruster_t200_from_yaml name="thruster_vsa" value="${thruster_data['vector_stbd_aft])}"/>
+    <!-- Create Thrusters -->
+    <xacro:uuv_thruster_t200_from_yaml data="${thruster_data['heave_port_fwd']}"/>
+    <xacro:uuv_thruster_t200_from_yaml data="${thruster_data['heave_port_aft']}"/>
+    <xacro:uuv_thruster_t200_from_yaml data="${thruster_data['heave_stbd_fwd']}"/>
+    <xacro:uuv_thruster_t200_from_yaml data="${thruster_data['heave_stbd_aft']}"/>
+    <xacro:uuv_thruster_t200_from_yaml data="${thruster_data['vector_port_fwd']}"/>
+    <xacro:uuv_thruster_t200_from_yaml data="${thruster_data['vector_port_aft']}"/>
+    <xacro:uuv_thruster_t200_from_yaml data="${thruster_data['vector_stbd_fwd']}"/>
+    <xacro:uuv_thruster_t200_from_yaml data="${thruster_data['vector_stbd_aft']}"/>
 </robot>
