Commit message: URDF builds. Having dependency issues with gazebo/uuv_sim.

File: common_robot_description/xacro/common_joints.xacro (robot description, xacro)
@@ -1,4 +1,4 @@
 <?xml version="1.0"?>
-<robot xmlns:xacro="http://www.ros.org/wiki/xacro" name="common_links">
+<robot xmlns:xacro="http://www.ros.org/wiki/xacro" name="common_joint_macros">
   <xacro:include filename="$(find common_robot_description)/xacro/common_tags.xacro"/>
   <xacro:property name="tag_axis" value="axis"/>

File: common_robot_description/xacro/common_links.xacro (robot description, xacro)
@@ -1,5 +1,6 @@
 <?xml version="1.0"?>
-<robot xmlns:xacro="http://www.ros.org/wiki/xacro" name="common_links">
+<robot xmlns:xacro="http://www.ros.org/wiki/xacro" name="common_link_macros">
   <xacro:include filename="$(find common_robot_description)/xacro/common_tags.xacro"/>
+  <xacro:include filename="$(find uuv_gazebo_ros_plugins)/urdf/snippets.xacro"/>
   <!-- Link Tags -->
   <xacro:property name="tag_collision" value="collision"/>
@@ -131,5 +132,5 @@
   <xacro:macro name="uuv_hydro_links" params="flow_topic:='hydrodynamics/current_velocity' fluid_density:=1000 **uuv_links">
     <gazebo>
-      <plugin name="uuv_plugin" filename="libuuv_underwater_object_ros_plugin.so">
+      <plugin filename="libuuv_underwater_object_ros_plugin.so" name="uuv_plugin">
         <fluid_density>${fluid_density}</fluid_density>
         <flow_velocity_topic>${flow_topic}</flow_velocity_topic>

File: common_robot_description/xacro/common_thrusters.xacro (robot description, xacro)
@@ -1,7 +1,8 @@
 <?xml version="1.0"?>
-<robot xmlns:xacro="http://www.ros.org/wiki/xacro" name="common_thrusters">
+<robot xmlns:xacro="http://www.ros.org/wiki/xacro" name="common_thruster_macros">
   <xacro:include filename="$(find common_robot_description)/xacro/common_tags.xacro"/>
   <xacro:include filename="$(find common_robot_description)/xacro/common_links.xacro"/>
   <xacro:include filename="$(find common_robot_description)/xacro/common_joints.xacro"/>
+  <xacro:include filename="$(find uuv_gazebo_ros_plugins)/urdf/snippets.xacro"/>
   <!-- Thruster Tags -->
   <xacro:property name="tag_thrust" value="thrust"/>
@@ -21,30 +22,4 @@
     <xacro:standard_link_from_yaml name="${data[tag_link][tag_name]}" data="${t200[tag_link]}"/>
     <xacro:standard_joint_from_yaml data="${data[tag_joint]}" child="${data[tag_link][tag_name]}"/>
-    <!--<link name="${data[tag_link][tag_name]}">
-      <visual>
-        <geometry>
-          <mesh filename="${t200_data[tag_link][tag_mesh]}" scale="1 1 1" />
-        </geometry>
-      </visual>
-      <inertial>
-        <mass value="${t200_data[tag_link][tag_mass]}" />
-        <origin xyz="${t200_data[tag_link][tag_com][tag_x]} ${t200_data[tag_link][tag_com][tag_y]} ${t200_data[tag_link][tag_com][tag_z]}"
-                rpy="0 0 0"/>
-        <inertia ixx="${t200_data[tag_link][tag_inertia][tag_ixx]}"
-                ixy="${t200_data[tag_link][tag_inertia][tag_ixy]}"
-                ixz="${t200_data[tag_link][tag_inertia][tag_ixz]}"
-                iyy="${t200_data[tag_link][tag_inertia][tag_iyy]}"
-                iyz="${t200_data[tag_link][tag_inertia][tag_iyz]}"
-                izz="${t200_data[tag_link][tag_inertia][tag_izz]}" />
-      </inertial>
-    </link>-->
-    <!-- Joint between thruster link and vehicle base link -->
-    <!--<joint name="${data[tag_joint][tag_name]}" type="continuous">
-      <origin xyz="${data[tag_joint][tag_origin][tag_xyz]}"
-              rpy="${data[tag_joint][tag_origin][tag_rpy]}"/>
-      <axis xyz="${data[tag_joint][tag_axis]}" />
-      <parent link="${data[tag_joint][tag_parent]}" />
-      <child link="${data[tag_link][tag_name]}" />
-    </joint>-->
     <gazebo>
       <plugin name="thruster_model_${data[tag_thruster][tag_name]}" filename="libuuv_thruster_ros_plugin.so">

File: maelstrom_description/model/robots/maelstrom.urdf.xacro (robot description, xacro)
@@ -15,9 +15,16 @@
   <!-- Combine hydro links -->
   <!-- Can add more within uuv_links as the model grows -->
-  <xacro:uuv_hydro_links>
+  <!--<xacro:uuv_hydro_links>
     <uuv_links>
       <xacro:maelstrom_base_uuv_links/>
     </uuv_links>
-  </xacro:uuv_hydro_links>
+  </xacro:uuv_hydro_links>-->
+  <gazebo>
+    <plugin name="uuv_underwater_object_ros_plugin" filename="libuuv_underwater_object_ros_plugin.so">
+      <fluid_density>1028</fluid_density>
+      <flow_velocity_topic>hydrodynamic/current_velocity</flow_velocity_topic>
+      <xacro:maelstrom_base_uuv_links/>
+    </plugin>
+  </gazebo>
   <!-- Joint state publisher plugin -->
   <xacro:default_joint_state_publisher namespace="$(arg namespace)" update_rate="10"/>

File: maelstrom_description/model/xacro/sensors.xacro (robot description, xacro)
@@ -63,5 +63,5 @@
 				namespace="${namespace}"
 				parent_link="base_link"
-				inertial_reference_frame="world_ned">
+				inertial_reference_frame="world">
 				<origin xyz="0 0 0" rpy="0 0 0"/>
 	</xacro:default_imu_macro>
