Commit message: Added common sensors macros. Almost done

File: common_robot_description/xacro/common_joints.xacro (robot description, xacro)
@@ -1,17 +1,17 @@
 <?xml version="1.0"?>
 <robot xmlns:xacro="http://www.ros.org/wiki/xacro" name="common_joint_macros">
-  <xacro:include filename="$(find common_robot_description)/xacro/common_tags.xacro"/>
-  <xacro:property name="tag_axis" value="axis"/>
-  <xacro:property name="tag_damping" value="damping"/>
-  <xacro:property name="tag_dynamics" value="dynamics"/>
-  <xacro:property name="tag_parent" value="parent"/>
-  <xacro:macro name="standard_joint_from_yaml" params="name:=None data child">
-   <joint name="${data[tag_name] if name is None else name}" type="${data[tag_type]}">
-      <origin xyz="${data[tag_origin][tag_xyz]}"
-              rpy="${data[tag_origin][tag_rpy]}"/>
-      <axis xyz="${data[tag_axis]}" />
-      <parent link="${data[tag_parent]}" />
-      <child link="${child}" />
-    </joint>
-  </xacro:macro>
+   <xacro:include filename="$(find common_robot_description)/xacro/common_tags.xacro"/>
+   <xacro:property name="tag_axis" value="axis"/>
+   <xacro:property name="tag_damping" value="damping"/>
+   <xacro:property name="tag_dynamics" value="dynamics"/>
+   <xacro:property name="tag_parent" value="parent"/>
+   <xacro:macro name="standard_joint_from_yaml" params="name:=None data child">
+      <joint name="${data[tag_name] if name is None else name}" type="${data[tag_type]}">
+         <origin xyz="${data[tag_origin][tag_xyz]}"
+                  rpy="${data[tag_origin][tag_rpy]}"/>
+         <axis xyz="${data[tag_axis]}" />
+         <parent link="${data[tag_parent]}" />
+         <child link="${child}" />
+      </joint>
+   </xacro:macro>
 </robot>

File: common_robot_description/xacro/common_links.xacro (robot description, xacro)
@@ -1,141 +1,132 @@
 <?xml version="1.0"?>
 <robot xmlns:xacro="http://www.ros.org/wiki/xacro" name="common_link_macros">
-  <xacro:include filename="$(find common_robot_description)/xacro/common_tags.xacro"/>
-  <xacro:include filename="$(find uuv_gazebo_ros_plugins)/urdf/snippets.xacro"/>
-  <!-- Link Tags -->
-  <xacro:property name="tag_collision" value="collision"/>
-  <xacro:property name="tag_com" value="com"/>
-  <xacro:property name="tag_dummy_joint" value="dummy_joint"/>
-  <xacro:property name="tag_dummy_link" value="dummy_link"/>
-  <xacro:property name="tag_inertia" value="inertia"/>
-  <xacro:property name="tag_ixx" value="ixx"/>
-  <xacro:property name="tag_ixy" value="ixy"/>
-  <xacro:property name="tag_ixz" value="ixz"/>
-  <xacro:property name="tag_iyy" value="iyy"/>
-  <xacro:property name="tag_iyz" value="iyz"/>
-  <xacro:property name="tag_izz" value="izz"/>
-  <xacro:property name="tag_mass" value="mass"/>
-  <xacro:property name="tag_mesh" value="mesh_properties"/>
-  <xacro:property name="tag_visual" value="visual"/>
-  <!-- Hydro Link Tags -->
-  <xacro:property name="tag_added_mass" value="added_mass"/>
-  <xacro:property name="tag_box" value="box"/>
-  <xacro:property name="tag_constant" value="constant"/>
-  <xacro:property name="tag_cob" value="cob"/>
-  <xacro:property name="tag_damping" value="damping"/>
-  <xacro:property name="tag_height" value="height"/>
-  <xacro:property name="tag_hydro" value="hydro"/>
-  <xacro:property name="tag_length" value="length"/>
-  <xacro:property name="tag_linear" value="linear"/>
-  <xacro:property name="tag_quadratic" value="quadratic"/>
-  <xacro:property name="tag_volume" value="volume"/>
-  <xacro:property name="tag_width" value="width"/>
-  <xacro:macro name="inertia_from_yaml" params="data">
-    <inertia ixx="${data[tag_ixx]}" ixy="${data[tag_ixy]}" ixz="${data[tag_ixz]}"
-             iyy="${data[tag_iyy]}" iyz="${data[tag_iyz]}" izz="${data[tag_izz]}"/>
-  </xacro:macro>
-  <xacro:macro name="base_link_from_yaml" params="data">
-    <link name="${data[tag_name]}">
-      <xacro:if value="${tag_mesh in data}">
-        <xacro:if value="${tag_visual in data[tag_mesh]}">
-          <visual>
-            <geometry>
-              <mesh filename="${data[tag_mesh][tag_visual]}" scale="1 1 1"/>
-            </geometry>
-            <origin xyz="0.0 0.0 0.0" rpy="0.0 0.0 0.0"/>
-          </visual>
-        </xacro:if>
-        <xacro:if value="${tag_collision in data[tag_mesh]}">
-          <visual>
-            <geometry>
-              <mesh filename="${data[tag_mesh][tag_collision]}" scale="1 1 1"/>
-            </geometry>
-            <origin xyz="0.0 0.0 0.0" rpy="0.0 0.0 0.0"/>
-          </visual>
-        </xacro:if>
-      </xacro:if>
-    </link>
-    <link name="${data[tag_dummy_link][tag_name]}">
-      <inertial>
-        <mass value="${data[tag_mass]}"/>
-        <origin xyz="${data[tag_com][tag_x]} ${data[tag_com][tag_y]} ${data[tag_com][tag_z]}" rpy="0 0 0"/>
-        <inertia ixx="${data[tag_inertia][tag_ixx]}"
-                ixy="${data[tag_inertia][tag_ixy]}"
-                ixz="${data[tag_inertia][tag_ixz]}"
-                iyy="${data[tag_inertia][tag_iyy]}"
-                iyz="${data[tag_inertia][tag_iyz]}"
-                izz="${data[tag_inertia][tag_izz]}" />
-      </inertial>
-    </link>
-    <joint name="${data[tag_dummy_joint][tag_name]}" type="fixed">
-      <parent link="${data[tag_name]}"/>
-      <child link="${data[tag_dummy_link][tag_name]}"/>
-    </joint>
-    <gazebo reference="${data[tag_name]}">
-      <selfCollide>false</selfCollide>
-    </gazebo>
-  </xacro:macro>
-  <xacro:macro name="standard_link_from_yaml" params="name:=None data">
-    <link name="${data[tag_name] if name is None else name}">
-      <xacro:if value="${tag_mesh in data}">
-        <xacro:if value="${tag_visual in data[tag_mesh]}">
-          <visual>
-            <geometry>
-              <mesh filename="${data[tag_mesh][tag_visual]}" scale="1 1 1"/>
-            </geometry>
-            <origin xyz="0.0 0.0 0.0" rpy="0.0 0.0 0.0"/>
-          </visual>
-        </xacro:if>
-        <xacro:if value="${tag_collision in data[tag_mesh]}">
-          <visual>
-            <geometry>
-              <mesh filename="${data[tag_mesh][tag_collision]}" scale="1 1 1"/>
-            </geometry>
-            <origin xyz="0.0 0.0 0.0" rpy="0.0 0.0 0.0"/>
-          </visual>
-        </xacro:if>
-      </xacro:if>
-      <inertial>
-        <mass value="${data[tag_mass]}"/>
-        <origin xyz="${data[tag_com][tag_x]} ${data[tag_com][tag_y]} ${data[tag_com][tag_z]}" rpy="0 0 0"/>
-        <inertia ixx="${data[tag_inertia][tag_ixx]}"
-                ixy="${data[tag_inertia][tag_ixy]}"
-                ixz="${data[tag_inertia][tag_ixz]}"
-                iyy="${data[tag_inertia][tag_iyy]}"
-                iyz="${data[tag_inertia][tag_iyz]}"
-                izz="${data[tag_inertia][tag_izz]}" />
-      </inertial>
-    </link>
-  </xacro:macro>
-  <xacro:macro name="hydro_link_from_yaml" params="name data">
-    <link name="${name}">
-      <volume>${data[tag_volume]}</volume>
-      <!-- Link's bounding box, it is used to recalculate the immersed
-      volume when close to the surface.
-      This is a workaround the invalid bounding box given by Gazebo-->
-      <xacro:if value="${tag_box in data}">
-        <box>
-          <width>${data[tag_box][tag_width]}</width>
-          <length>${data[tag_box][tag_length]}</length>
-          <height>${data[tag_box][tag_height]}</height>
-        </box>
-      </xacro:if>
-      <center_of_buoyancy>${data[tag_cob]}</center_of_buoyancy> <!-- In the body frame -->
-      <hydrodynamic_model>
-        <type>fossen</type>
-        <added_mass>${data[tag_added_mass]}</added_mass>
-        <linear_damping>${data[tag_damping][tag_linear]}</linear_damping>
-        <quadratic_damping>${data[tag_damping][tag_quadratic]}</quadratic_damping>
-      </hydrodynamic_model>
-    </link>
-  </xacro:macro>
-  <xacro:macro name="uuv_hydro_links" params="flow_topic:='hydrodynamics/current_velocity' fluid_density:=1000 **uuv_links">
-    <gazebo>
-      <plugin filename="libuuv_underwater_object_ros_plugin.so" name="uuv_plugin">
-        <fluid_density>${fluid_density}</fluid_density>
-        <flow_velocity_topic>${flow_topic}</flow_velocity_topic>
-        <xacro:insert_block name="uuv_links"/>
-      </plugin>
-    </gazebo>
-  </xacro:macro>
+   <xacro:include filename="$(find common_robot_description)/xacro/common_tags.xacro"/>
+   <xacro:include filename="$(find uuv_gazebo_ros_plugins)/urdf/snippets.xacro"/>
+   <!-- Link Tags -->
+   <xacro:property name="tag_collision" value="collision"/>
+   <xacro:property name="tag_com" value="com"/>
+   <xacro:property name="tag_dummy_joint" value="dummy_joint"/>
+   <xacro:property name="tag_dummy_link" value="dummy_link"/>
+   <xacro:property name="tag_inertial" value="inertial"/>
+   <xacro:property name="tag_inertia" value="inertia"/>
+   <xacro:property name="tag_ixx" value="ixx"/>
+   <xacro:property name="tag_ixy" value="ixy"/>
+   <xacro:property name="tag_ixz" value="ixz"/>
+   <xacro:property name="tag_iyy" value="iyy"/>
+   <xacro:property name="tag_iyz" value="iyz"/>
+   <xacro:property name="tag_izz" value="izz"/>
+   <xacro:property name="tag_mass" value="mass"/>
+   <xacro:property name="tag_mesh" value="mesh_properties"/>
+   <xacro:property name="tag_visual" value="visual"/>
+   <!-- Hydro Link Tags -->
+   <xacro:property name="tag_added_mass" value="added_mass"/>
+   <xacro:property name="tag_box" value="box"/>
+   <xacro:property name="tag_constant" value="constant"/>
+   <xacro:property name="tag_cob" value="cob"/>
+   <xacro:property name="tag_damping" value="damping"/>
+   <xacro:property name="tag_height" value="height"/>
+   <xacro:property name="tag_hydro" value="hydro"/>
+   <xacro:property name="tag_length" value="length"/>
+   <xacro:property name="tag_linear" value="linear"/>
+   <xacro:property name="tag_quadratic" value="quadratic"/>
+   <xacro:property name="tag_volume" value="volume"/>
+   <xacro:property name="tag_width" value="width"/>
+   <xacro:macro name="inertia_from_yaml" params="data">
+      <inertia ixx="${data[tag_ixx]}" ixy="${data[tag_ixy]}" ixz="${data[tag_ixz]}"
+               iyy="${data[tag_iyy]}" iyz="${data[tag_iyz]}" izz="${data[tag_izz]}"/>
+   </xacro:macro>
+   <xacro:macro name="origin_from_yaml" params="data">
+      <origin xyz="${data[tag_xyz]}" rpy="${data[tag_rpy]}"/>
+   </xacro:macro>
+   <xacro:macro name="inertial_from_yaml" params="data">
+      <mass value="${data[tag_mass]}"/>
+      <xacro:inertia_from_yaml data="${data[tag_inertia]}"/>
+      <origin xyz="${data[tag_com]}" rpy="0 0 0"/>
+   </xacro:macro>
+   <xacro:macro name="base_link_from_yaml" params="data">
+      <link name="${data[tag_name]}">
+         <xacro:if value="${tag_mesh in data}">
+            <xacro:if value="${tag_visual in data[tag_mesh]}">
+               <visual>
+                  <geometry>
+                     <mesh filename="${data[tag_mesh][tag_visual]}" scale="1 1 1"/>
+                  </geometry>
+                  <origin xyz="0 0 0" rpy="0 0 0"/>
+               </visual>
+            </xacro:if>
+            <xacro:if value="${tag_collision in data[tag_mesh]}">
+               <visual>
+                  <geometry>
+                     <mesh filename="${data[tag_mesh][tag_collision]}" scale="1 1 1"/>
+                  </geometry>
+                  <origin xyz="0 0 0" rpy="0 0 0"/>
+               </visual>
+            </xacro:if>
+         </xacro:if>
+      </link>
+      <link name="${data[tag_dummy_link][tag_name]}">
+         <xacro:inertial_from_yaml data="${data[tag_inertial]}"/>
+      </link>
+      <joint name="${data[tag_dummy_joint][tag_name]}" type="fixed">
+         <parent link="${data[tag_name]}"/>
+         <child link="${data[tag_dummy_link][tag_name]}"/>
+      </joint>
+      <gazebo reference="${data[tag_name]}">
+         <selfCollide>false</selfCollide>
+      </gazebo>
+   </xacro:macro>
+   <xacro:macro name="standard_link_from_yaml" params="name:=None data">
+      <link name="${data[tag_name] if name is None else name}">
+         <xacro:if value="${tag_mesh in data}">
+            <xacro:if value="${tag_visual in data[tag_mesh]}">
+               <visual>
+                  <geometry>
+                     <mesh filename="${data[tag_mesh][tag_visual]}" scale="1 1 1"/>
+                  </geometry>
+                  <origin xyz="0 0 0" rpy="0 0 0"/>
+               </visual>
+            </xacro:if>
+            <xacro:if value="${tag_collision in data[tag_mesh]}">
+               <visual>
+                  <geometry>
+                     <mesh filename="${data[tag_mesh][tag_collision]}" scale="1 1 1"/>
+                  </geometry>
+                  <origin xyz="0 0 0" rpy="0 0 0"/>
+               </visual>
+            </xacro:if>
+         </xacro:if>
+         <xacro:inertial_from_yaml data="${data[tag_inertial]}"/>
+      </link>
+   </xacro:macro>
+   <xacro:macro name="hydro_link_from_yaml" params="name data">
+      <link name="${name}">
+         <volume>${data[tag_volume]}</volume>
+         <!-- Link's bounding box, it is used to recalculate the immersed
+         volume when close to the surface.
+         This is a workaround the invalid bounding box given by Gazebo-->
+         <xacro:if value="${tag_box in data}">
+            <box>
+               <width>${data[tag_box][tag_width]}</width>
+               <length>${data[tag_box][tag_length]}</length>
+               <height>${data[tag_box][tag_height]}</height>
+            </box>
+         </xacro:if>
+         <center_of_buoyancy>${data[tag_cob][tag_x]} ${data[tag_cob][tag_y]} ${data[tag_cob][tag_z]}</center_of_buoyancy> <!-- In the body frame -->
+         <hydrodynamic_model>
+            <type>fossen</type>
+            <added_mass>${data[tag_added_mass]}</added_mass>
+            <linear_damping>${data[tag_damping][tag_linear]}</linear_damping>
+            <quadratic_damping>${data[tag_damping][tag_quadratic]}</quadratic_damping>
+         </hydrodynamic_model>
+      </link>
+   </xacro:macro>
+   <xacro:macro name="uuv_hydro_links" params="flow_topic:='hydrodynamics/current_velocity' fluid_density:=1000 **uuv_links">
+      <gazebo>
+         <plugin filename="libuuv_underwater_object_ros_plugin.so" name="uuv_underwater_object_ros_plugin">
+            <fluid_density>${fluid_density}</fluid_density>
+            <flow_velocity_topic>${flow_topic}</flow_velocity_topic>
+            <xacro:insert_block name="uuv_links"/>
+         </plugin>
+      </gazebo>
+   </xacro:macro>
 </robot>

File: common_robot_description/xacro/common_thrusters.xacro (robot description, xacro)
@@ -27,5 +27,4 @@
         <jointName>${data[tag_joint][tag_name]}</jointName>
         <thrusterID>${data[tag_thruster][tag_id]}</thrusterID>
-        <!-- Minimum and maximum thrust force output allowed -->
         <thrustMax>${t200[tag_limits][tag_thrust][tag_max]}</thrustMax>
         <thrustMin>${t200[tag_limits][tag_thrust][tag_min]}</thrustMin>
@@ -38,5 +37,4 @@
         Function: thrust = rotorConstant * x * abs(x)
         -->
-        <!-- TODO: Find good thruster model -->
         <conversion>
           <type>${t200[tag_gazebo][tag_conversion][tag_type]}</type>

File: maelstrom_description/model/robots/maelstrom.urdf.xacro (robot description, xacro)
@@ -1,31 +1,24 @@
 <?xml version="1.0"?>
 <robot name="maelstrom" xmlns:xacro="http://www.ros.org/wiki/xacro" >
-  <xacro:arg name="debug" default="0"/>
-  <xacro:arg name="namespace" default="maelstrom"/>
-  <xacro:property name="namespace" value="$(arg namespace)"/>
-  <!-- Include common xacros -->
-  <xacro:include filename="$(find uuv_descriptions)/urdf/common.urdf.xacro"/>
-  <xacro:include filename="$(find common_robot_description)/xacro/common_tags.xacro"/>
-  <xacro:include filename="$(find common_robot_description)/xacro/common_links.xacro"/>
-  <xacro:include filename="$(find common_robot_description)/xacro/common_joints.xacro"/>
-  <!-- Create Maelstrom -->
-  <xacro:include filename="$(find maelstrom_description)/model/xacro/base.xacro"/>
-  <xacro:include filename="$(find maelstrom_description)/model/xacro/thrusters.xacro"/>
-  <xacro:include filename="$(find maelstrom_description)/model/xacro/sensors.xacro"/>
-  <!-- Combine hydro links -->
-  <!-- Can add more within uuv_links as the model grows -->
-  <!--<xacro:uuv_hydro_links>
-    <uuv_links>
-      <xacro:maelstrom_base_uuv_links/>
-    </uuv_links>
-  </xacro:uuv_hydro_links>-->
-  <gazebo>
-    <plugin name="uuv_underwater_object_ros_plugin" filename="libuuv_underwater_object_ros_plugin.so">
-      <fluid_density>1028</fluid_density>
-      <flow_velocity_topic>hydrodynamic/current_velocity</flow_velocity_topic>
-      <xacro:maelstrom_base_uuv_links/>
-    </plugin>
-  </gazebo>
-  <!-- Joint state publisher plugin -->
-  <xacro:default_joint_state_publisher namespace="$(arg namespace)" update_rate="10"/>
+	<xacro:arg name="debug" default="0"/>
+	<xacro:arg name="namespace" default="maelstrom"/>
+	<xacro:property name="namespace" value="$(arg namespace)"/>
+	<!-- Include common xacros -->
+	<xacro:include filename="$(find uuv_descriptions)/urdf/common.urdf.xacro"/>
+	<xacro:include filename="$(find common_robot_description)/xacro/common_tags.xacro"/>
+	<xacro:include filename="$(find common_robot_description)/xacro/common_links.xacro"/>
+	<xacro:include filename="$(find common_robot_description)/xacro/common_joints.xacro"/>
+	<!-- Create Maelstrom -->
+	<xacro:include filename="$(find maelstrom_description)/model/xacro/base.xacro"/>
+	<xacro:include filename="$(find maelstrom_description)/model/xacro/thrusters.xacro"/>
+	<xacro:include filename="$(find maelstrom_description)/model/xacro/sensors.xacro"/>
+	<!-- Combine hydro links -->
+	<!-- Can add more within uuv_links as the model grows -->
+	<xacro:uuv_hydro_links>
+	   <uuv_links>
+		   <xacro:maelstrom_base_uuv_hydro_links/>
+	   </uuv_links>
+	</xacro:uuv_hydro_links>
+	<!-- Joint state publisher plugin -->
+	<xacro:default_joint_state_publisher namespace="$(arg namespace)" update_rate="10"/>
 </robot>

File: maelstrom_description/model/xacro/base.xacro (robot description, xacro)
@@ -8,5 +8,5 @@
   <xacro:property name="base" value="${base_data['base_link']}"/>
   <xacro:base_link_from_yaml data="${base[tag_link]}"/>
-  <xacro:macro name="maelstrom_base_uuv_links">
+  <xacro:macro name="maelstrom_base_uuv_hydro_links">
     <xacro:hydro_link_from_yaml name="${base[tag_link][tag_name]}" data="${base[tag_link][tag_hydro]}"/>
   </xacro:macro>

File: maelstrom_description/model/xacro/sensors.xacro (robot description, xacro)
@@ -1,79 +1,13 @@
 <?xml version="1.0"?>
-<robot xmlns:xacro="http://www.ros.org/wiki/xacro">
-	<xacro:include filename="$(find uuv_sensor_ros_plugins)/urdf/sensor_snippets.xacro"/>
-	<xacro:property name="forward_camera_R_pos"><origin xyz="0.3818 0.05038 0.11999" rpy="0 0 0" /></xacro:property>
-    <xacro:property name="forward_camera_L_pos"><origin xyz="0.3818 -0.05038 0.11999" rpy="0 0 0" /></xacro:property>
-    <xacro:property name="downward_camera_pos"><origin xyz="0.0711 0.0004 0" rpy="0 ${pi/2} 0" /></xacro:property>
-  <!--
-    Some examples of sensors that can be added to the vehicle frame.
-    Set the origin of the sensor frames correctly for your application
-    Look into the sensor macros in the package uuv_sensor_ros_plugins/urdf for
-    more examples or add you own custom sensor units.
-  -->
-	<!-- right forward camerea-->
-	<xacro:regular_camera_plugin_macro
-				namespace="sensors"
-				suffix="_forward_R"
-				parent_link="base_link"
-				topic="camera"
-				mass="0.001"
-				update_rate="30"
-				hfov="1.5125"
-				width="768"
-				height="492"
-				stddev="0.02"
-				scale="1.0">
-				<inertia ixx="0.00001" ixy="0.0" ixz="0.0" iyy="0.00001" iyz="0.0" izz="0.00001" />
-				<xacro:insert_block name="forward_camera_R_pos" />
-	</xacro:regular_camera_plugin_macro>
-	<!-- left forward camera-->
-	<xacro:regular_camera_plugin_macro
-				namespace="sensors"
-				suffix="_forward_L"
-				parent_link="base_link"
-				topic="camera"
-				mass="0.001"
-				update_rate="30"
-				hfov="1.5125"
-				width="768"
-				height="492"
-				stddev="0.02"
-				scale="1.0">
-				<inertia ixx="0.00001" ixy="0.0" ixz="0.0" iyy="0.00001" iyz="0.0" izz="0.00001" />
-				<xacro:insert_block name="forward_camera_L_pos" />
-	</xacro:regular_camera_plugin_macro>
-	<!-- downward camera-->
-	<xacro:regular_camera_plugin_macro
-				namespace="sensors"
-				suffix="_downward"
-				parent_link="base_link"
-				topic="camera"
-				mass="0.001"
-				update_rate="30"
-				hfov="1.5125"
-				width="768"
-				height="492"
-				stddev="0.02"
-				scale="1.0">
-				<inertia ixx="0.00001" ixy="0.0" ixz="0.0" iyy="0.00001" iyz="0.0" izz="0.00001" />
-				<xacro:insert_block name="downward_camera_pos" />
-	</xacro:regular_camera_plugin_macro>
-	<!-- IMU -->
-	<xacro:default_imu_macro
-				namespace="${namespace}"
-				parent_link="base_link"
-				inertial_reference_frame="world">
-				<origin xyz="0 0 0" rpy="0 0 0"/>
-	</xacro:default_imu_macro>
-	<!--DVL-->
-	<xacro:default_dvl_macro
-				namespace="${namespace}"
-				parent_link="base_link"
-				inertial_reference_frame="world_ned">
-				<origin xyz="-0.081297 -0.081297 0.0" rpy="0 ${0.5*pi} 0"/>
-	</xacro:default_dvl_macro>
-	<!--Depth Sensor-->
-	<xacro:default_pressure_macro namespace="${namespace}" parent_link="base_link">
-				<origin xyz="0 -0.0004 0.0711" rpy="0 0 0"/>
-	</xacro:default_pressure_macro>
+<robot xmlns:xacro="http://www.ros.org/wiki/xacro" name="sensors">
+	<xacro:include filename="$(find common_robot_description)/xacro/common_sensors.xacro"/>
+	<!-- Load data from yaml -->
+   <xacro:property name="sensors_file" value="$(find maelstrom_description)/model/config/sensors.yaml"/>
+   <xacro:property name="sensors_data" value="${load_yaml(sensors_file)}"/>
+   <xacro:camera_from_yaml data="${sensors_file['camera']['forward_R']}"/>
+   <xacro:camera_from_yaml data="${sensors_file['camera']['forward_L']}"/>
+   <xacro:camera_from_yaml data="${sensors_file['camera']['downward']}"/>
+   <xacro:depth_from_yaml data="${sensors_file['depth']['depth']}"/>
+   <xacro:imu_from_yaml data="${sensors_file['imu']['imu']}"/>
+   <xacro:dvl_from_yaml data="${sensors_file['dvl']['dvl']}"/>
 </robot>
