Commit message: Added common sensors macros. Almost done

File: maelstrom_description/model/xacro/thrusters.xacro (robot description, xacro)
@@ -1,18 +1,18 @@
 <?xml version="1.0"?>
 <robot xmlns:xacro="http://www.ros.org/wiki/xacro" name="thrusters">
-    <!-- Include needed xacros -->
-    <xacro:include filename="$(find uuv_gazebo_ros_plugins)/urdf/snippets.xacro"/>
-    <xacro:include filename="$(find common_robot_description)/xacro/common_thrusters.xacro"/>
-    <!-- Load data from yaml -->
-    <xacro:property name="thruster_file" value="$(find maelstrom_description)/model/config/thrusters.yaml"/>
-    <xacro:property name="thruster_data" value="${load_yaml(thruster_file)}"/>
-    <!-- Create Thrusters -->
-    <xacro:uuv_thruster_t200_from_yaml data="${thruster_data['heave_port_fwd']}"/>
-    <xacro:uuv_thruster_t200_from_yaml data="${thruster_data['heave_port_aft']}"/>
-    <xacro:uuv_thruster_t200_from_yaml data="${thruster_data['heave_stbd_fwd']}"/>
-    <xacro:uuv_thruster_t200_from_yaml data="${thruster_data['heave_stbd_aft']}"/>
-    <xacro:uuv_thruster_t200_from_yaml data="${thruster_data['vector_port_fwd']}"/>
-    <xacro:uuv_thruster_t200_from_yaml data="${thruster_data['vector_port_aft']}"/>
-    <xacro:uuv_thruster_t200_from_yaml data="${thruster_data['vector_stbd_fwd']}"/>
-    <xacro:uuv_thruster_t200_from_yaml data="${thruster_data['vector_stbd_aft']}"/>
+   <!-- Include needed xacros -->
+   <xacro:include filename="$(find uuv_gazebo_ros_plugins)/urdf/snippets.xacro"/>
+   <xacro:include filename="$(find common_robot_description)/xacro/common_thrusters.xacro"/>
+   <!-- Load data from yaml -->
+   <xacro:property name="thruster_file" value="$(find maelstrom_description)/model/config/thrusters.yaml"/>
+   <xacro:property name="thruster_data" value="${load_yaml(thruster_file)}"/>
+   <!-- Create Thrusters -->
+   <xacro:uuv_thruster_t200_from_yaml data="${thruster_data['heave_port_fwd']}"/>
+   <xacro:uuv_thruster_t200_from_yaml data="${thruster_data['heave_port_aft']}"/>
+   <xacro:uuv_thruster_t200_from_yaml data="${thruster_data['heave_stbd_fwd']}"/>
+   <xacro:uuv_thruster_t200_from_yaml data="${thruster_data['heave_stbd_aft']}"/>
+   <xacro:uuv_thruster_t200_from_yaml data="${thruster_data['vector_port_fwd']}"/>
+   <xacro:uuv_thruster_t200_from_yaml data="${thruster_data['vector_port_aft']}"/>
+   <xacro:uuv_thruster_t200_from_yaml data="${thruster_data['vector_stbd_fwd']}"/>
+   <xacro:uuv_thruster_t200_from_yaml data="${thruster_data['vector_stbd_aft']}"/>
 </robot>

Commit message: Finished yaml config for xacro

File: common_robot_description/xacro/common_joints.xacro (robot description, xacro)
@@ -10,7 +10,7 @@
          <origin xyz="${data[tag_origin][tag_xyz]}"
                   rpy="${data[tag_origin][tag_rpy]}"/>
-         <axis xyz="${data[tag_axis]}" />
-         <parent link="${data[tag_parent]}" />
-         <child link="${child}" />
+         <axis xyz="${data[tag_axis]}"/>
+         <parent link="${data[tag_parent]}"/>
+         <child link="${child}"/>
       </joint>
    </xacro:macro>

File: common_robot_description/xacro/common_links.xacro (robot description, xacro)
@@ -40,7 +40,9 @@
    </xacro:macro>
    <xacro:macro name="inertial_from_yaml" params="data">
-      <mass value="${data[tag_mass]}"/>
-      <xacro:inertia_from_yaml data="${data[tag_inertia]}"/>
-      <origin xyz="${data[tag_com]}" rpy="0 0 0"/>
+      <inertial>
+         <mass value="${data[tag_mass]}"/>
+         <xacro:inertia_from_yaml data="${data[tag_inertia]}"/>
+         <origin xyz="${data[tag_com]}" rpy="0 0 0"/>
+      </inertial>
    </xacro:macro>
    <xacro:macro name="base_link_from_yaml" params="data">
@@ -112,5 +114,5 @@
             </box>
          </xacro:if>
-         <center_of_buoyancy>${data[tag_cob][tag_x]} ${data[tag_cob][tag_y]} ${data[tag_cob][tag_z]}</center_of_buoyancy> <!-- In the body frame -->
+         <center_of_buoyancy>${data[tag_cob]}</center_of_buoyancy> <!-- Relative to CoM -->
          <hydrodynamic_model>
             <type>fossen</type>

File: common_robot_description/xacro/common_sensors.xacro (robot description, xacro)
@@ -16,43 +16,34 @@
    <xacro:property name="tag_topic" value="topic"/>
    <xacro:property name="tag_width" value="width"/>
-   <xacro:macro name="camera_from_yaml" params="namespace:=sensors topic:=camera_ data">
-      <xacro:regular_camera_plugin_macro
-         	namespace="${namespace}"
-            suffix="${data[tag_suffix]}"
-            parent_link="${data[tag_parent]}"
-            topic="${topic}"
-            mass="${data[tag_mass]}"
-            update_rate="${data[tag_rate]}"
-            hfov="${data[tag_hfov]}"
-            width="${data[tag_width]}"
-            height="${data[tag_height]}"
-            stddev="${data[tag_stddev]}"
-            scale="${data[tag_scale]}">
-            <xacro:inertia_from_yaml data="${data[tag_inertia]}" />
-            <xacro:origin_from_yam; name="${data[tag_origin]}" />
+   <xacro:macro name="camera_from_yaml" params="namespace:=sensors topic:=camera data">
+      <xacro:regular_camera_plugin_macro namespace="${namespace}"
+                                          suffix="${data[tag_suffix]}"
+                                          parent_link="${data[tag_parent]}"
+                                          topic="${topic}"
+                                          mass="${data[tag_mass]}"
+                                          update_rate="${data[tag_rate]}"
+                                          hfov="${data[tag_hfov]}"
+                                          width="${data[tag_width]}"
+                                          height="${data[tag_height]}"
+                                          stddev="${data[tag_stddev]}"
+                                          scale="${data[tag_scale]}">
+         <xacro:inertia_from_yaml data="${data[tag_inertia]}" />
+         <xacro:origin_from_yaml data="${data[tag_origin]}" />
       </xacro:regular_camera_plugin_macro>
    </xacro:macro>
    <xacro:macro name="pressure_from_yaml" params="namespace:=sensors data">
-      <xacro:default_pressure_macro
-               namespace="${namespace}"
-               parent_link="${data[tag_parent]}">
-               <xacro:origin_from_yaml data="$data[tag_origin]}"/>
+      <xacro:default_pressure_macro namespace="${namespace}" parent_link="${data[tag_parent]}">
+         <xacro:origin_from_yaml data="${data[tag_origin]}"/>
       </xacro:default_pressure_macro>
    </xacro:macro>
    <xacro:macro name="imu_from_yaml" params="namespace:=sensors data">
-      <xacro:default_imu_macro
-               namespace="${namespace}"
-               parent_link="${data[tag_parent]}"
-               inertial_reference_frame="${data[tag_ref_frame]}">
-               <xacro:origin_from_yaml data="$data[tag_origin]}"/>
+      <xacro:default_imu_macro namespace="${namespace}" parent_link="${data[tag_parent]}" inertial_reference_frame="${data[tag_ref_frame]}">
+         <xacro:origin_from_yaml data="${data[tag_origin]}"/>
       </xacro:default_imu_macro>
    </xacro:macro>
    <xacro:macro name="dvl_from_yaml" params="namespace:=sensors data">
-      <xacro:default_dvl_macro
-               namespace="${namespace}"
-               parent_link="${data[tag_parent]}"
-               inertial_reference_frame="${data[tag_ref_frame]}">
-               <xacro:origin_from_yaml data="$data[tag_origin]}"/>
-      </xacro:default_imu_macro>
+      <xacro:default_dvl_macro namespace="${namespace}" parent_link="${data[tag_parent]}" inertial_reference_frame="${data[tag_ref_frame]}">
+         <xacro:origin_from_yaml data="${data[tag_origin]}"/>
+      </xacro:default_dvl_macro>
    </xacro:macro>
 </robot>

File: common_robot_description/xacro/common_thrusters.xacro (robot description, xacro)
@@ -23,5 +23,5 @@
     <xacro:standard_joint_from_yaml data="${data[tag_joint]}" child="${data[tag_link][tag_name]}"/>
     <gazebo>
-      <plugin name="thruster_model_${data[tag_thruster][tag_name]}" filename="libuuv_thruster_ros_plugin.so">
+      <plugin name="${data[tag_link][tag_name]}_model" filename="libuuv_thruster_ros_plugin.so">
         <linkName>${data[tag_link][tag_name]}</linkName>
         <jointName>${data[tag_joint][tag_name]}</jointName>

File: maelstrom_description/model/xacro/sensors.xacro (robot description, xacro)
@@ -5,9 +5,9 @@
    <xacro:property name="sensors_file" value="$(find maelstrom_description)/model/config/sensors.yaml"/>
    <xacro:property name="sensors_data" value="${load_yaml(sensors_file)}"/>
-   <xacro:camera_from_yaml data="${sensors_file['camera']['forward_R']}"/>
-   <xacro:camera_from_yaml data="${sensors_file['camera']['forward_L']}"/>
-   <xacro:camera_from_yaml data="${sensors_file['camera']['downward']}"/>
-   <xacro:depth_from_yaml data="${sensors_file['depth']['depth']}"/>
-   <xacro:imu_from_yaml data="${sensors_file['imu']['imu']}"/>
-   <xacro:dvl_from_yaml data="${sensors_file['dvl']['dvl']}"/>
+   <xacro:camera_from_yaml data="${sensors_data['camera']['forward_R']}"/>
+   <xacro:camera_from_yaml data="${sensors_data['camera']['forward_L']}"/>
+   <xacro:camera_from_yaml data="${sensors_data['camera']['downward']}"/>
+   <xacro:pressure_from_yaml data="${sensors_data['depth']['depth']}"/>
+   <xacro:imu_from_yaml data="${sensors_data['imu']['imu']}"/>
+   <xacro:dvl_from_yaml data="${sensors_data['dvl']['dvl']}"/>
 </robot>

Commit message: Getting it all working and cleaned up

File: common_robot_description/xacro/common_joints.xacro (robot description, xacro)
@@ -7,5 +7,5 @@
    <xacro:property name="tag_parent" value="parent"/>
    <xacro:macro name="standard_joint_from_yaml" params="name:=None data child">
-      <joint name="${data[tag_name] if name is None else name}" type="${data[tag_type]}">
+      <joint name="${data[tag_name]}" type="${data[tag_type]}">
          <origin xyz="${data[tag_origin][tag_xyz]}"
                   rpy="${data[tag_origin][tag_rpy]}"/>

File: common_robot_description/xacro/common_links.xacro (robot description, xacro)
@@ -58,10 +58,10 @@
             </xacro:if>
             <xacro:if value="${tag_collision in data[tag_mesh]}">
-               <visual>
+               <collision>
                   <geometry>
                      <mesh filename="${data[tag_mesh][tag_collision]}" scale="1 1 1"/>
                   </geometry>
                   <origin xyz="0 0 0" rpy="0 0 0"/>
-               </visual>
+               </collision>
             </xacro:if>
          </xacro:if>

File: common_robot_description/xacro/common_thrusters.xacro (robot description, xacro)
@@ -18,8 +18,7 @@
     Dummy link as place holder for the thruster frame,
     since thrusters can often be inside the collision geometry
-    of the vehicle and may cause internal collisions if set otherwise
-    -->
+    of the vehicle and may cause internal collisions if set otherwise-->
     <xacro:standard_link_from_yaml name="${data[tag_link][tag_name]}" data="${T200[tag_link]}"/>
-    <xacro:standard_joint_from_yaml data="${data[tag_joint]}" child="${data[tag_link][tag_name]}"/>
+    <xacro:standard_joint_from_yaml name="${data[tag_joint][tag_name]}" data="${data[tag_joint]}" child="${data[tag_link][tag_name]}"/>
     <gazebo>
       <plugin name="${data[tag_link][tag_name]}_model" filename="libuuv_thruster_ros_plugin.so">
