Commit message: Revised sensors config

File: common_robot_description/xacro/common_sensors.xacro (robot description, xacro)
@@ -6,7 +6,9 @@
    <xacro:property name="tag_height" value="height"/>
    <xacro:property name="tag_hfov" value="hfov"/>
-   <xacro:property name="tag_ref_frame" value="inertial_reference_frame"/>
+   <xacro:property name="tag_ref_frame" value="reference_frame"/>
    <xacro:property name="tag_namespace" value="namesapce"/>
    <xacro:property name="tag_mass" value="mass"/>
+   <xacro:property name="tag_noise_amplitude" value="noise_amplitude"/>
+   <xacro:property name="tag_noise_sigma" value="noise_sigma"/>
    <xacro:property name="tag_parent" value="parent_link"/>
    <xacro:property name="tag_rate" value="update_rate"/>
@@ -21,5 +23,5 @@
                                           parent_link="${data[tag_parent]}"
                                           topic="${topic}"
-                                          mass="${data[tag_mass]}"
+                                          mass="0.01"
                                           update_rate="${data[tag_rate]}"
                                           hfov="${data[tag_hfov]}"
@@ -28,22 +30,44 @@
                                           stddev="${data[tag_stddev]}"
                                           scale="${data[tag_scale]}">
-         <xacro:inertia_from_yaml data="${data[tag_inertia]}" />
+         <inertia ixx="0.01" ixy="0" ixz="0" iyy="0.01" iyz="0" izz="0.01"/>
          <xacro:origin_from_yaml data="${data[tag_origin]}" />
       </xacro:regular_camera_plugin_macro>
    </xacro:macro>
-   <xacro:macro name="pressure_from_yaml" params="namespace:=sensors data">
-      <xacro:default_pressure_macro namespace="${namespace}" parent_link="${data[tag_parent]}">
+   <xacro:macro name="pressure_from_yaml" params="namespace:=sensors topic:=pressure data">
+      <xacro:pressure_plugin_macro  namespace="${namespace}"
+                                    suffix="${data[tag_suffix]}"
+                                    parent_link="${data[tag_parent]}"
+                                    topic="${topic}"
+                                    mass="0.015"
+                                    update_rate="${data[tag_rate]}"
+                                    range="30000"
+                                    noise_sigma="${data[tag_noise_sigma]}"
+                                    noise_amplitude="${data[tag_noise_amplitude]}"
+                                    estimateDepth="false"
+                                    standardPressure="101.325"
+                                    kPaPerM="9.80638">
+         <inertia ixx="0.001" ixy="0" ixz="0" iyy="0.001" iyz="0" izz="0.001"/>
          <xacro:origin_from_yaml data="${data[tag_origin]}"/>
-      </xacro:default_pressure_macro>
+      </xacro:pressure_plugin_macro>
    </xacro:macro>
-   <xacro:macro name="imu_from_yaml" params="namespace:=sensors data">
-      <xacro:default_imu_macro namespace="${namespace}" parent_link="${data[tag_parent]}" inertial_reference_frame="${data[tag_ref_frame]}">
+   <xacro:macro name="imu_from_yaml" params="namespace:=sensors topic:=imu data">
+      <xacro:default_imu_macro namespace="${namespace}"
+                               parent_link="${data[tag_parent]}"
+                               inertial_reference_frame="${data[tag_ref_frame]}">
          <xacro:origin_from_yaml data="${data[tag_origin]}"/>
       </xacro:default_imu_macro>
    </xacro:macro>
-   <xacro:macro name="dvl_from_yaml" params="namespace:=sensors data">
-      <xacro:default_dvl_macro namespace="${namespace}" parent_link="${data[tag_parent]}" inertial_reference_frame="${data[tag_ref_frame]}">
+   <xacro:macro name="dvl_from_yaml" params="namespace:=sensors topic:=dvl data">
+      <xacro:dvl_plugin_macro namespace="${namespace}"
+                              suffix="${data[tag_suffix]}"
+                              parent_link="${data[tag_parent]}"
+                              reference_frame="${data[tag_ref_frame]}"
+                              update_rate="${data[tag_rate]}"
+                              topic="${topic}"
+                              noise_sigma="${data[tag_noise_sigma]}"
+                              noise_amplitude="${data[tag_noise_amplitude]}"
+                              scale="1">
          <xacro:origin_from_yaml data="${data[tag_origin]}"/>
-      </xacro:default_dvl_macro>
+      </xacro:dvl_plugin_macro>
    </xacro:macro>
 </robot>

File: maelstrom_description/model/xacro/sensors.xacro (robot description, xacro)
@@ -8,5 +8,5 @@
    <xacro:camera_from_yaml data="${sensors_data['camera']['forward_L']}"/>
    <xacro:camera_from_yaml data="${sensors_data['camera']['downward']}"/>
-   <xacro:pressure_from_yaml data="${sensors_data['depth']['depth']}"/>
+   <xacro:pressure_from_yaml data="${sensors_data['pressure']['pressure']}"/>
    <xacro:imu_from_yaml data="${sensors_data['imu']['imu']}"/>
    <xacro:dvl_from_yaml data="${sensors_data['dvl']['dvl']}"/>

Commit message: Adding stereo

File: common_robot_description/xacro/common_sensors.xacro (robot description, xacro)
@@ -1,72 +1,173 @@
-<?xml version="1.0"?>
+<?xml version="1.0" ?>
 <robot xmlns:xacro="http://www.ros.org/wiki/xacro" name="common_sensor_macros">
-   <xacro:include filename="$(find uuv_sensor_ros_plugins)/urdf/sensor_snippets.xacro"/>
-   <xacro:include filename="$(find common_robot_description)/xacro/common_links.xacro"/>
+   <xacro:include filename="$(find uuv_sensor_ros_plugins)/urdf/sensor_snippets.xacro" />
+   <xacro:include filename="$(find common_robot_description)/xacro/common_links.xacro" />
    <!-- Sensor Tags -->
-   <xacro:property name="tag_height" value="height"/>
-   <xacro:property name="tag_hfov" value="hfov"/>
-   <xacro:property name="tag_ref_frame" value="reference_frame"/>
-   <xacro:property name="tag_namespace" value="namesapce"/>
-   <xacro:property name="tag_mass" value="mass"/>
-   <xacro:property name="tag_noise_amplitude" value="noise_amplitude"/>
-   <xacro:property name="tag_noise_sigma" value="noise_sigma"/>
-   <xacro:property name="tag_parent" value="parent_link"/>
-   <xacro:property name="tag_rate" value="update_rate"/>
-   <xacro:property name="tag_scale" value="scale"/>
-   <xacro:property name="tag_stddev" value="stddev"/>
-   <xacro:property name="tag_suffix" value="topic_suffix"/>
-   <xacro:property name="tag_topic" value="topic"/>
-   <xacro:property name="tag_width" value="width"/>
+   <xacro:property name="tag_height" value="height" />
+   <xacro:property name="tag_hfov" value="hfov" />
+   <xacro:property name="tag_ref_frame" value="reference_frame" />
+   <xacro:property name="tag_namespace" value="namesapce" />
+   <xacro:property name="tag_mass" value="mass" />
+   <xacro:property name="tag_noise_amplitude" value="noise_amplitude" />
+   <xacro:property name="tag_noise_sigma" value="noise_sigma" />
+   <xacro:property name="tag_parent" value="parent_link" />
+   <xacro:property name="tag_rate" value="update_rate" />
+   <xacro:property name="tag_scale" value="scale" />
+   <xacro:property name="tag_stddev" value="stddev" />
+   <xacro:property name="tag_suffix" value="topic_suffix" />
+   <xacro:property name="tag_topic" value="topic" />
+   <xacro:property name="tag_width" value="width" />
    <xacro:macro name="camera_from_yaml" params="namespace:=sensors topic:=camera data">
-      <xacro:regular_camera_plugin_macro namespace="${namespace}"
-                                          suffix="${data[tag_suffix]}"
-                                          parent_link="${data[tag_parent]}"
-                                          topic="${topic}"
-                                          mass="0.01"
-                                          update_rate="${data[tag_rate]}"
-                                          hfov="${data[tag_hfov]}"
-                                          width="${data[tag_width]}"
-                                          height="${data[tag_height]}"
-                                          stddev="${data[tag_stddev]}"
-                                          scale="${data[tag_scale]}">
-         <inertia ixx="0.01" ixy="0" ixz="0" iyy="0.01" iyz="0" izz="0.01"/>
+      <xacro:regular_camera_plugin_macro namespace="${namespace}" suffix="${data[tag_suffix]}" parent_link="${data[tag_parent]}" topic="${topic}"
+      mass="0.01" update_rate="${data[tag_rate]}" hfov="${data[tag_hfov]}" width="${data[tag_width]}" height="${data[tag_height]}"
+      stddev="${data[tag_stddev]}" scale="${data[tag_scale]}">
+         <inertia ixx="0.01" ixy="0" ixz="0" iyy="0.01" iyz="0" izz="0.01" />
          <xacro:origin_from_yaml data="${data[tag_origin]}" />
       </xacro:regular_camera_plugin_macro>
    </xacro:macro>
+   <xacro:macro name="stereo_from_yaml" params="namespace:=stereo topic:=camera data">
+      <xacro:property name="k1l" value="0" />
+      <xacro:property name="k2l" value="0" />
+      <xacro:property name="p1l" value="0" />
+      <xacro:property name="p2l" value="0" />
+      <xacro:property name="k3l" value="0" />
+      <xacro:property name="k1r" value="0" />
+      <xacro:property name="k2r" value="0" />
+      <xacro:property name="p1r" value="0" />
+      <xacro:property name="p2r" value="0" />
+      <xacro:property name="k3r" value="0" />
+      <xacro:property name="hfov" value="${data[tag_hfov]}" />
+      <link name="${namespace}/stereo_left_link">
+         <inertial>
+            <mass value=".001" />
+            <inertia ixx="0" ixy="0.0" ixz="0.0" iyy="0" iyz="0.0" izz="0" />
+         </inertial>
+         <xacro:no_collision />
+      </link>
+      <joint name="${namespace}/stereo_joint" type="revolute">
+         <xacro:origin_from_yaml data="${data[tag_origin]}" />
+         <parent link="${data[tag_parent]}" />
+         <child link="${namespace}/stereo_left_link" />
+         <limit upper="0" lower="0" effort="0" velocity="0" />
+         <axis xyz="1 0 0" />
+      </joint>
+      <gazebo reference="${namespace}/stereo_left_link">
+         <sensor name="camera" type="camera">
+            <camera>
+               <horizontal_fov>${hfov}</horizontal_fov>
+               <image>
+                  <width>${data[tag_width]}</width>
+                  <height>${data[tag_height]}</height>
+                  <format>R8G8B8</format>
+               </image>
+               <clip>
+                  <near>0.05</near>
+                  <far>5000</far>
+               </clip>
+               <noise>
+                  <type>gaussian</type>
+                  <mean>0.0</mean>
+                  <stddev>${data[tag_stddev]}</stddev>
+                </noise>
+               <distortion>
+                  <k1>${k1l}</k1>
+                  <k2>${k2l}</k2>
+                  <k3>${k3l}</k3>
+                  <p1>${p1l}</p1>
+                  <p2>${p2l}</p2>
+                  <center>0.5 0.5</center>
+               </distortion>
+            </camera>
+            <plugin name="left_controller" filename="libgazebo_ros_camera.so">
+               <alwaysOn>true</alwaysOn>
+               <updateRate>${data[tag_rate]}</updateRate>
+               <cameraName>${namespace}/left</cameraName>
+               <imageTopicName>image_raw</imageTopicName>
+               <cameraInfoTopicName>camera_info</cameraInfoTopicName>
+               <frameName>${namespace}/stereo_left_link</frameName>
+               <distortionK1>${k1l}</distortionK1>
+               <distortionK2>${k2l}</distortionK2>
+               <distortionK3>${k3l}</distortionK3>
+               <distortionT1>${p1l}</distortionT1>
+               <distortionT2>${p2l}</distortionT2>
+            </plugin>
+            <always_on>1</always_on>
+            <update_rate>${data[tag_rate]}</update_rate>
+         </sensor>
+      </gazebo>
+      <link name="${namespace}/stereo_right_link">
+         <inertial>
+            <mass value="0.01" />
+            <inertia ixx="0" ixy="0.0" ixz="0.0" iyy="0" iyz="0.0" izz="0" />
+         </inertial>
+         <xacro:no_collision />
+      </link>
+      <joint name="${namespace}/stereo_right_joint" type="revolute">
+         <origin xyz="0.0 -0.1 0" rpy="0 0 0" />
+         <parent link="${namespace}/stereo_left_link" />
+         <child link="${namespace}/stereo_right_link" />
+         <limit upper="0" lower="0" effort="0" velocity="0" />
+         <axis xyz="1 0 0" />
+      </joint>
+      <gazebo reference="${namespace}/stereo_right_link">
+         <sensor name="camera" type="camera">
+            <camera>
+               <horizontal_fov>${hfov}</horizontal_fov>
+               <image>
+                  <width>${data[tag_width]}</width>
+                  <height>${data[tag_height]}</height>
+                  <format>R8G8B8</format>
+               </image>
+               <clip>
+                  <near>0.05</near>
+                  <far>5000</far>
+               </clip>
+               <noise>
+                  <type>gaussian</type>
+                  <mean>0.0</mean>
+                  <stddev>${data[tag_stddev]}</stddev>
+                </noise>
+               <distortion>
+                  <k1>${k1l}</k1>
+                  <k2>${k2l}</k2>
+                  <k3>${k3l}</k3>
+                  <p1>${p1l}</p1>
+                  <p2>${p2l}</p2>
+                  <center>0.5 0.5</center>
+               </distortion>
+            </camera>
+            <plugin name="right_controller" filename="libgazebo_ros_camera.so">
+               <alwaysOn>true</alwaysOn>
+               <updateRate>${data[tag_rate]}</updateRate>
+               <cameraName>${namespace}/right</cameraName>
+               <imageTopicName>image_raw</imageTopicName>
+               <cameraInfoTopicName>camera_info</cameraInfoTopicName>
+               <frameName>${namespace}/stereo_right_link</frameName>
+               <hackBaseline>0.1</hackBaseline>
+               <distortionK1>${k1l}</distortionK1>
+               <distortionK2>${k2l}</distortionK2>
+               <distortionK3>${k3l}</distortionK3>
+               <distortionT1>${p1l}</distortionT1>
+               <distortionT2>${p2l}</distortionT2>
+            </plugin>
+            <always_on>1</always_on>
+            <update_rate>${data[tag_rate]}</update_rate>
+         </sensor>
+      </gazebo>
+   </xacro:macro>
    <xacro:macro name="pressure_from_yaml" params="namespace:=sensors topic:=pressure data">
-      <xacro:pressure_plugin_macro  namespace="${namespace}"
-                                    suffix="${data[tag_suffix]}"
-                                    parent_link="${data[tag_parent]}"
-                                    topic="${topic}"
-                                    mass="0.015"
-                                    update_rate="${data[tag_rate]}"
-                                    range="30000"
-                                    noise_sigma="${data[tag_noise_sigma]}"
-                                    noise_amplitude="${data[tag_noise_amplitude]}"
-                                    estimateDepth="false"
-                                    standardPressure="101.325"
-                                    kPaPerM="9.80638">
-         <inertia ixx="0.001" ixy="0" ixz="0" iyy="0.001" iyz="0" izz="0.001"/>
-         <xacro:origin_from_yaml data="${data[tag_origin]}"/>
+      <xacro:pressure_plugin_macro namespace="${namespace}" suffix="${data[tag_suffix]}" parent_link="${data[tag_parent]}" topic="${topic}" mass="0.015" update_rate="${data[tag_rate]}" range="30000" noise_sigma="${data[tag_noise_sigma]}" noise_amplitude="${data[tag_noise_amplitude]}" estimateDepth="false" standardPressure="101.325" kPaPerM="9.80638">
+         <inertia ixx="0.001" ixy="0" ixz="0" iyy="0.001" iyz="0" izz="0.001" />
+         <xacro:origin_from_yaml data="${data[tag_origin]}" />
       </xacro:pressure_plugin_macro>
    </xacro:macro>
    <xacro:macro name="imu_from_yaml" params="namespace:=sensors topic:=imu data">
-      <xacro:default_imu_macro namespace="${namespace}"
-                               parent_link="${data[tag_parent]}"
-                               inertial_reference_frame="${data[tag_ref_frame]}">
-         <xacro:origin_from_yaml data="${data[tag_origin]}"/>
+      <xacro:default_imu_macro namespace="${namespace}" parent_link="${data[tag_parent]}" inertial_reference_frame="${data[tag_ref_frame]}">
+         <xacro:origin_from_yaml data="${data[tag_origin]}" />
       </xacro:default_imu_macro>
    </xacro:macro>
    <xacro:macro name="dvl_from_yaml" params="namespace:=sensors topic:=dvl data">
-      <xacro:dvl_plugin_macro namespace="${namespace}"
-                              suffix="${data[tag_suffix]}"
-                              parent_link="${data[tag_parent]}"
-                              reference_frame="${data[tag_ref_frame]}"
-                              update_rate="${data[tag_rate]}"
-                              topic="${topic}"
-                              noise_sigma="${data[tag_noise_sigma]}"
-                              noise_amplitude="${data[tag_noise_amplitude]}"
-                              scale="1">
-         <xacro:origin_from_yaml data="${data[tag_origin]}"/>
+      <xacro:dvl_plugin_macro namespace="${namespace}" suffix="${data[tag_suffix]}" parent_link="${data[tag_parent]}" reference_frame="${data[tag_ref_frame]}" update_rate="${data[tag_rate]}" topic="${topic}" noise_sigma="${data[tag_noise_sigma]}" noise_amplitude="${data[tag_noise_amplitude]}" scale="1">
+         <xacro:origin_from_yaml data="${data[tag_origin]}" />
       </xacro:dvl_plugin_macro>
    </xacro:macro>

File: puddles_description/urdf/sensors.xacro (robot description, xacro)
@@ -5,6 +5,5 @@
    <xacro:property name="sensors_file" value="$(find puddles_description)/config/sensors.yaml"/>
    <xacro:property name="sensors_data" value="${load_yaml(sensors_file)}"/>
-   <xacro:camera_from_yaml data="${sensors_data['camera']['forward_R']}"/>
-   <xacro:camera_from_yaml data="${sensors_data['camera']['forward_L']}"/>
+   <xacro:stereo_from_yaml data="${sensors_data['camera']['stereo']}"/>
    <xacro:camera_from_yaml data="${sensors_data['camera']['downward']}"/>
    <!-- Only an IMU is needed among the inertial sensors, but all are included to represent the actual vehicle -->

Commit message: Fining sensor positions

File: common_robot_description/xacro/common_sensors.xacro (robot description, xacro)
@@ -45,10 +45,14 @@
          <xacro:no_collision />
       </link>
-      <joint name="${namespace}/stereo_joint" type="revolute">
+      <joint name="${namespace}/stereo_left_joint" type="fixed">
          <xacro:origin_from_yaml data="${data[tag_origin]}" />
          <parent link="${data[tag_parent]}" />
          <child link="${namespace}/stereo_left_link" />
-         <limit upper="0" lower="0" effort="0" velocity="0" />
-         <axis xyz="1 0 0" />
+      </joint>
+      <link name="${namespace}/stereo_left_optical" />
+      <joint name="${namespace}/stereo_left_optical_joint" type="fixed">
+         <parent link="${namespace}/stereo_left_link" />
+         <child link="${namespace}/stereo_left_optical" />
+         <origin rpy="-1.570796 0 -1.570796"></origin>
       </joint>
       <gazebo reference="${namespace}/stereo_left_link">
@@ -85,5 +89,5 @@
                <imageTopicName>image_raw</imageTopicName>
                <cameraInfoTopicName>camera_info</cameraInfoTopicName>
-               <frameName>${namespace}/stereo_left_link</frameName>
+               <frameName>${namespace}/stereo_left_optical</frameName>
                <distortionK1>${k1l}</distortionK1>
                <distortionK2>${k2l}</distortionK2>
@@ -103,10 +107,14 @@
          <xacro:no_collision />
       </link>
-      <joint name="${namespace}/stereo_right_joint" type="revolute">
+      <joint name="${namespace}/stereo_right_joint" type="fixed">
          <origin xyz="0.0 -0.1 0" rpy="0 0 0" />
          <parent link="${namespace}/stereo_left_link" />
          <child link="${namespace}/stereo_right_link" />
-         <limit upper="0" lower="0" effort="0" velocity="0" />
-         <axis xyz="1 0 0" />
+      </joint>
+      <link name="${namespace}/stereo_right_optical" />
+      <joint name="${namespace}/stereo_right_optical_joint" type="fixed">
+         <parent link="${namespace}/stereo_right_link" />
+         <child link="${namespace}/stereo_right_optical" />
+         <origin rpy="-1.570796 0 -1.570796"></origin>
       </joint>
       <gazebo reference="${namespace}/stereo_right_link">
@@ -143,5 +151,5 @@
                <imageTopicName>image_raw</imageTopicName>
                <cameraInfoTopicName>camera_info</cameraInfoTopicName>
-               <frameName>${namespace}/stereo_right_link</frameName>
+               <frameName>${namespace}/stereo_right_optical</frameName>
                <hackBaseline>0.1</hackBaseline>
                <distortionK1>${k1l}</distortionK1>
