Commit message: Renaming maelstrom and removing pole

File: puddles_description/urdf/base.xacro (robot description, xacro)
@@ -3,10 +3,10 @@
   <xacro:include filename="$(find common_robot_description)/xacro/common_tags.xacro"/>
   <xacro:include filename="$(find common_robot_description)/xacro/common_links.xacro"/>
-  <!-- Load Maelstrom Base Data -->
-  <xacro:property name="base_file" value="$(find maelstrom_description)/config/base.yaml"/>
+  <!-- Load puddles Base Data -->
+  <xacro:property name="base_file" value="$(find puddles_description)/config/base.yaml"/>
   <xacro:property name="base_data" value="${load_yaml(base_file)}"/>
   <xacro:property name="base" value="${base_data['base_link']}"/>
   <xacro:base_link_from_yaml data="${base[tag_link]}"/>
-  <xacro:macro name="maelstrom_base_uuv_hydro_links">
+  <xacro:macro name="puddles_base_uuv_hydro_links">
     <xacro:hydro_link_from_yaml name="${base[tag_link][tag_name]}" data="${base[tag_link][tag_hydro]}"/>
   </xacro:macro>

File: puddles_description/urdf/puddles.urdf.xacro (robot description, xacro)
@@ -1,6 +1,6 @@
 <?xml version="1.0"?>
-<robot name="maelstrom" xmlns:xacro="http://www.ros.org/wiki/xacro" >
+<robot name="puddles" xmlns:xacro="http://www.ros.org/wiki/xacro" >
 	<xacro:arg name="debug" default="0"/>
-	<xacro:arg name="namespace" default="maelstrom"/>
+	<xacro:arg name="namespace" default="puddles"/>
 	<xacro:property name="namespace" value="$(arg namespace)"/>
 	<!-- Include common xacros -->
@@ -9,13 +9,13 @@
 	<xacro:include filename="$(find common_robot_description)/xacro/common_links.xacro"/>
 	<xacro:include filename="$(find common_robot_description)/xacro/common_joints.xacro"/>
-	<!-- Create Maelstrom -->
-	<xacro:include filename="$(find maelstrom_description)/urdf/base.xacro"/>
-	<xacro:include filename="$(find maelstrom_description)/urdf/thrusters.xacro"/>
-	<xacro:include filename="$(find maelstrom_description)/urdf/sensors.xacro"/>
+	<!-- Create puddles -->
+	<xacro:include filename="$(find puddles_description)/urdf/base.xacro"/>
+	<xacro:include filename="$(find puddles_description)/urdf/thrusters.xacro"/>
+	<xacro:include filename="$(find puddles_description)/urdf/sensors.xacro"/>
 	<!-- Combine hydro links -->
 	<!-- Can add more within uuv_links as the model grows -->
 	<xacro:uuv_hydro_links>
 	   <uuv_links>
-		   <xacro:maelstrom_base_uuv_hydro_links/>
+		   <xacro:puddles_base_uuv_hydro_links/>
 	   </uuv_links>
 	</xacro:uuv_hydro_links>

File: puddles_description/urdf/sensors.xacro (robot description, xacro)
@@ -3,5 +3,5 @@
 	<xacro:include filename="$(find common_robot_description)/xacro/common_sensors.xacro"/>
 	<!-- Load data from yaml -->
-   <xacro:property name="sensors_file" value="$(find maelstrom_description)/config/sensors.yaml"/>
+   <xacro:property name="sensors_file" value="$(find puddles_description)/config/sensors.yaml"/>
    <xacro:property name="sensors_data" value="${load_yaml(sensors_file)}"/>
    <xacro:camera_from_yaml data="${sensors_data['camera']['forward_R']}"/>

File: puddles_description/urdf/thrusters.xacro (robot description, xacro)
@@ -5,5 +5,5 @@
    <xacro:include filename="$(find common_robot_description)/xacro/common_thrusters.xacro"/>
    <!-- Load data from yaml -->
-   <xacro:property name="thruster_file" value="$(find maelstrom_description)/config/thrusters.yaml"/>
+   <xacro:property name="thruster_file" value="$(find puddles_description)/config/thrusters.yaml"/>
    <xacro:property name="thruster_data" value="${load_yaml(thruster_file)}"/>
    <!-- Create Thrusters -->
