Commit message: Fix inertia bug and downward camera

File: riptide_descriptions/urdf/snippets.xacro (robot description, xacro)
@@ -4,6 +4,6 @@
   <xacro:macro name="dummy_inertia">
     <inertial>
-      <mass value=".001" />
-      <inertia ixx="0" ixy="0.0" ixz="0.0" iyy="0" iyz="0.0" izz="0" />
+      <mass value=".0001" />
+      <inertia ixx="0.0001" ixy="0.0" ixz="0.0" iyy="0.0001" iyz="0.0" izz="0.0001" />
     </inertial>
   </xacro:macro>
