Commit message: Everything seems to work

File: riptide_descriptions/robots/puddles_default.xacro (robot description, xacro)
@@ -6,5 +6,4 @@
   <!-- Include the ROV macro file -->
   <xacro:include filename="$(find riptide_descriptions)/urdf/robot_base.xacro"/>
-  <xacro:include filename="$(find riptide_descriptions)/urdf/puddles.gazebo.xacro"/>
   <xacro:property name="yaml_file" value="$(find riptide_descriptions)/config/puddles.yaml" />
   <xacro:property name="config" value="${load_yaml(yaml_file)}"/>
@@ -13,20 +12,6 @@
     namespace="$(arg namespace)"
     config="${config}"
-    inertial_reference_frame="$(arg inertial_reference_frame)">
-    <!--
-      The underwater object plugin is given as an input block parameter to
-      allow the addition of external models of manipulator units
-    -->
-    <gazebo>
-      <plugin name="uuv_plugin" filename="libuuv_underwater_object_ros_plugin.so">
-        <fluid_density>1028.0</fluid_density>
-        <flow_velocity_topic>hydrodynamics/current_velocity</flow_velocity_topic>
-        <debug>$(arg debug)</debug>
-        <!-- Adding the hydrodynamic and hydrostatic parameters for the vehicle-->
-        <xacro:puddles_hydro_model namespace="$(arg namespace)"/>
-      </plugin>
-    </gazebo>
-  </xacro:robot_base>
+    inertial_reference_frame="$(arg inertial_reference_frame)"/>
   <!-- Joint state publisher plugin -->
-  <xacro:default_joint_state_publisher namespace="$(arg namespace)" update_rate="50"/>
+  <xacro:default_joint_state_publisher namespace="$(arg namespace)" update_rate="200"/>
 </robot>

File: riptide_descriptions/urdf/robot.gazebo.xacro (robot description, xacro)
@@ -1,16 +1,10 @@
 <?xml version="1.0"?>
 <robot xmlns:xacro="http://www.ros.org/wiki/xacro">
-    <xacro:property name="cob" value="0.027 -0.008 0.036"/>
-    <xacro:property name="volume" value="0.041"/>
+    <xacro:property name="lin" value="${config['linear_damping']}"/>
+    <xacro:property name="quad" value="${config['quadratic_damping']}"/>
     <xacro:macro name="puddles_hydro_model" params="namespace">
         <link name="${namespace}/base_link">
-            <neutrally_buoyant>0</neutrally_buoyant>
-            <volume>${volume}</volume>
-            <box>
-                <width>0.89</width>
-                <length>0.5</length>
-                <height>0.33</height>
-            </box>
-            <center_of_buoyancy>${cob}</center_of_buoyancy>
+            <volume>${config['volume']}</volume>
+            <center_of_buoyancy>${config['cob'][0]-config['base_link'][0]} ${config['cob'][1]-config['base_link'][1]} ${config['cob'][2]-config['base_link'][2]}</center_of_buoyancy>
             <hydrodynamic_model>
                 <type>fossen</type>
@@ -24,8 +18,8 @@
                 </added_mass>
                 <linear_damping>
-                    -17.0 -50.0 -50.0 -4 -9 -9
+                    ${lin[0]} ${lin[1]} ${lin[2]} ${lin[3]} ${lin[4]} ${lin[5]}
                 </linear_damping>
                 <quadratic_damping>
-                    -180.0 -460.0 -460.0 -12 -24.0 -24.0
+                    ${quad[0]} ${quad[1]} ${quad[2]} ${quad[3]} ${quad[4]} ${quad[5]}
                 </quadratic_damping>
             </hydrodynamic_model>

File: riptide_descriptions/urdf/robot_base.xacro (robot description, xacro)
@@ -5,7 +5,8 @@
   <xacro:include filename="$(find uuv_sensor_ros_plugins)/urdf/sensor_snippets.xacro"/>
   <xacro:include filename="$(find riptide_descriptions)/urdf/snippets.xacro" />
+  <xacro:include filename="$(find riptide_descriptions)/urdf/robot.gazebo.xacro" />
   <xacro:include filename="$(find uuv_gazebo_ros_plugins)/urdf/snippets.xacro"/>
   <xacro:macro name="robot_base"
-    params="namespace config *gazebo inertial_reference_frame">
+    params="namespace config inertial_reference_frame">
     <!-- Due to uuv_sim, base_link must be near center of vehicle -->
     <link name="${namespace}/base_link"/>
@@ -43,7 +44,15 @@
     </joint>
     <!-- Set up hydrodynamic plugin given as input parameter -->
-    <xacro:insert_block name="gazebo"/>
+    <gazebo>
+      <plugin name="uuv_plugin" filename="libuuv_underwater_object_ros_plugin.so">
+        <fluid_density>1028.0</fluid_density>
+        <flow_velocity_topic>hydrodynamics/current_velocity</flow_velocity_topic>
+        <debug>$(arg debug)</debug>
+        <!-- Adding the hydrodynamic and hydrostatic parameters for the vehicle-->
+        <xacro:puddles_hydro_model namespace="$(arg namespace)"/>
+      </plugin>
+    </gazebo>
     <xacro:include filename="$(find riptide_descriptions)/urdf/robot_sensors.xacro" />
-    <!-- <xacro:include filename="$(find riptide_descriptions)/urdf/puddles_actuators.xacro" /> -->
+    <xacro:include filename="$(find riptide_descriptions)/urdf/robot_actuators.xacro" />
   </xacro:macro>
 </robot>

File: riptide_descriptions/urdf/robot_sensors.xacro (robot description, xacro)
@@ -28,5 +28,5 @@
       topic="${depth['topic']}"
       update_rate="${depth['rate']}"
-      range="30000"
+      range="300"
       noise_sigma="${depth['sigma']}"
       noise_amplitude="1"
@@ -66,7 +66,7 @@
     parent_link="${namespace}/base_link"
     inertial_reference_frame="${inertial_reference_frame}" />
-  <xacro:macro name="cameras_macro" params="namespace config">
-    <xacro:if value="${len(config)}">
-      <xacro:property name="camera" value="${config[0]}"/>
+  <xacro:macro name="cameras_macro" params="namespace cameras">
+    <xacro:if value="${len(cameras)}">
+      <xacro:property name="camera" value="${cameras[0]}"/>
       <xacro:if value="${camera['type'] == 'stereo'}">
         <xacro:stereo_macro
@@ -98,7 +98,7 @@
         </xacro:camera_macro>
       </xacro:unless>
-      <xacro:cameras_macro namespace="${namespace}" config="${config[1:]}"/>
+      <xacro:cameras_macro namespace="${namespace}" cameras="${cameras[1:]}"/>
     </xacro:if>
   </xacro:macro>
-  <xacro:cameras_macro namespace="${namespace}" config="${config['cameras']}"/>
+  <xacro:cameras_macro namespace="${namespace}" cameras="${config['cameras']}"/>
 </robot>

File: riptide_descriptions/urdf/snippets.xacro (robot description, xacro)
@@ -31,7 +31,7 @@
     <link name="${namespace}/${name}_optical" />
     <joint name="${namespace}/${name}_optical_joint" type="fixed">
-        <parent link="${namespace}/${name}_link" />
-        <child link="${namespace}/${name}_optical" />
-        <origin rpy="${-pi/2} 0 ${-pi/2}"></origin>
+      <parent link="${namespace}/${name}_link" />
+      <child link="${namespace}/${name}_optical" />
+      <origin rpy="${-pi/2} 0 ${-pi/2}"></origin>
     </joint>
     <gazebo reference="${namespace}/${name}_link">
@@ -285,3 +285,42 @@
     </gazebo>
   </xacro:macro>
+  <xacro:macro name="thruster_macro"
+    params="namespace
+            thruster_id
+            *origin
+            mesh_filename
+            rotor_constant">
+    <joint name="${namespace}/thruster_${thruster_id}_joint" type="continuous">
+      <xacro:insert_block name="origin"/>
+      <axis xyz="1 0 0"/>
+      <parent link="${namespace}/origin"/>
+      <child link="${namespace}/thruster_${thruster_id}"/>
+    </joint>
+    <link name="${namespace}/thruster_${thruster_id}">
+      <visual>
+        <geometry>
+          <mesh filename="${mesh_filename}" scale="1 1 1"/>
+        </geometry>
+      </visual>
+      <xacro:dummy_inertia />
+      <xacro:no_collision />
+    </link>
+    <gazebo>
+      <plugin name="${namespace}_${thruster_id}_thruster_model" filename="libuuv_thruster_ros_plugin.so">
+        <linkName>${namespace}/thruster_${thruster_id}</linkName>
+        <jointName>${namespace}/thruster_${thruster_id}_joint</jointName>
+        <thrusterID>${thruster_id}</thrusterID>
+        <dynamics>
+          <type>ZeroOrder</type>
+        </dynamics>
+        <conversion>
+          <type>Basic</type>
+          <rotorConstant>${rotor_constant}</rotorConstant>
+        </conversion>
+      </plugin>
+    </gazebo>
+    <gazebo reference="${namespace}/thruster_${thruster_id}">
+      <selfCollide>false</selfCollide>
+    </gazebo>
+  </xacro:macro>
 </robot>

Commit message: Cleanup and comments

File: riptide_descriptions/robots/puddles_default.xacro (robot description, xacro)
@@ -4,9 +4,10 @@
   <xacro:arg name="namespace" default="puddles"/>
   <xacro:arg name="inertial_reference_frame" default="world"/>
-  <!-- Include the ROV macro file -->
+  <!-- Include the Robot macro file -->
   <xacro:include filename="$(find riptide_descriptions)/urdf/robot_base.xacro"/>
+  <!-- Read the config -->
   <xacro:property name="yaml_file" value="$(find riptide_descriptions)/config/puddles.yaml" />
   <xacro:property name="config" value="${load_yaml(yaml_file)}"/>
-  <!-- Create puddles -->
+  <!-- Create robot -->
   <xacro:robot_base
     namespace="$(arg namespace)"

File: riptide_descriptions/urdf/robot.gazebo.xacro (robot description, xacro)
@@ -3,7 +3,9 @@
     <xacro:property name="lin" value="${config['linear_damping']}"/>
     <xacro:property name="quad" value="${config['quadratic_damping']}"/>
+    <!-- All hydro parameters for any links that have them -->
     <xacro:macro name="puddles_hydro_model" params="namespace">
         <link name="${namespace}/base_link">
             <volume>${config['volume']}</volume>
+            <!-- COB is relative to center of base_link, thus the math -->
             <center_of_buoyancy>${config['cob'][0]-config['base_link'][0]} ${config['cob'][1]-config['base_link'][1]} ${config['cob'][2]-config['base_link'][2]}</center_of_buoyancy>
             <hydrodynamic_model>

File: riptide_descriptions/urdf/robot_actuators.xacro (robot description, xacro)
@@ -13,4 +13,5 @@
 -->
 <robot xmlns:xacro="http://www.ros.org/wiki/xacro" >
+  <!-- Macro makes any number of thrusters from config -->
   <xacro:macro name="thrusters_macro" params="namespace config thrusters index">
     <xacro:if value="${len(thrusters)}">

File: riptide_descriptions/urdf/robot_base.xacro (robot description, xacro)
@@ -43,5 +43,5 @@
       <origin xyz="${config['com'][0]} ${config['com'][1]} ${config['com'][2]}" rpy="0 0 0"/>
     </joint>
-    <!-- Set up hydrodynamic plugin given as input parameter -->
+    <!-- Set up hydrodynamic plugin -->
     <gazebo>
       <plugin name="uuv_plugin" filename="libuuv_underwater_object_ros_plugin.so">

File: riptide_descriptions/urdf/robot_sensors.xacro (robot description, xacro)
@@ -39,4 +39,5 @@
   </xacro:if>
   <!-- IMU  -->
+  <!-- TODO: Get imu model from config -->
   <xacro:if value="${'imu' in config}">
     <xacro:property name="imu" value="${config['imu']}"/>
@@ -62,8 +63,10 @@
     </xacro:imu_plugin_macro>
   </xacro:if>
+  <!-- Pose sensor as ground truth for state estimation -->
   <xacro:default_pose_3d_macro
     namespace="${namespace}"
     parent_link="${namespace}/base_link"
     inertial_reference_frame="${inertial_reference_frame}" />
+  <!-- Builds any number of cameras from yaml -->
   <xacro:macro name="cameras_macro" params="namespace cameras">
     <xacro:if value="${len(cameras)}">

File: riptide_descriptions/urdf/snippets.xacro (robot description, xacro)
@@ -1,16 +1,5 @@
 <?xml version="1.0"?>
 <robot xmlns:xacro="http://www.ros.org/wiki/xacro" >
-  <!-- Thruster joint and link snippet -->
-  <xacro:macro name="thruster_macro"
-    params="namespace thruster_id *origin">
-    <xacro:thruster_module_first_order_basic_fcn_macro
-      namespace="${namespace}"
-      thruster_id="${thruster_id}"
-      mesh_filename="file://$(find riptide_descriptions)/meshes/Propeller.dae"
-      dyn_time_constant="0.05"
-      rotor_constant="0.026546960744430276">
-      <xacro:insert_block name="origin"/>
-    </xacro:thruster_module_first_order_basic_fcn_macro>
-  </xacro:macro>
+  <!-- Makes a blank inertia (gazebo needs this sometimes) -->
   <xacro:macro name="dummy_inertia">
     <inertial>
@@ -19,4 +8,5 @@
     </inertial>
   </xacro:macro>
+  <!-- TODO: Add camera distortion -->
   <xacro:macro name="camera_macro" params="namespace name parent_link update_rate hfov width height stddev baseline:=0 *origin">
     <link name="${namespace}/${name}_link">
@@ -191,5 +181,5 @@
         <sensor_topic>${topic}</sensor_topic> <!-- (string): name of the sensor output topic and prefix of service names -->
         <update_rate>${update_rate}</update_rate> <!-- Update period [s] -->
-        <noise_sigma>${noise_sigma}</noise_sigma> <!-- std dev of position estimates in x, y, z [m/s] -->
+        <noise_sigma>${noise_sigma}</noise_sigma> <!-- std dev of velocity estimates in x, y, z [m/s] -->
         <noise_amplitude>${noise_amplitude}</noise_amplitude>
         <enable_gazebo_messages>false</enable_gazebo_messages>
@@ -278,5 +268,5 @@
         <accelerometer_turn_on_bias_sigma>${accelerometer_turn_on_bias_sigma}</accelerometer_turn_on_bias_sigma> <!-- Accelerometer turn on bias standard deviation [m/s^2] -->
         <orientation_noise>${orientation_noise}</orientation_noise>
-        <update_rate>${update_rate}</update_rate> <!-- Update period of accelerometer and gyroscope [s] -->
+        <update_rate>${update_rate}</update_rate> <!-- Update frequency of accelerometer and gyroscope [s] -->
         <enable_gazebo_messages>false</enable_gazebo_messages>
         <enable_local_ned_frame>${enable_local_ned_frame}</enable_local_ned_frame>
